File: PCB/JayKey1.kicad_pcb (KiCad board)
At the start: 2 copper layers, 0 parts

Commit message: 2017.11.14 Update
- Redid schematic and layout
- Now using USB-C connector
Parts:
- added C_AVCC1: 100n, Capacitors_SMD:C_0805_HandSoldering, F.Cu at (297.7, 219.1)
- added C_CAP1: 1u, Capacitors_SMD:C_0805_HandSoldering, F.Cu at (302.4, 219.1)
- added C_CLK1: 22p, Capacitors_SMD:C_0805_HandSoldering, F.Cu at (307.2, 219.1)
- added C_CLK2: 22p, Capacitors_SMD:C_0805_HandSoldering, F.Cu at (311.9, 219.1)
- added C_REF1: 100n, Capacitors_SMD:C_0805_HandSoldering, F.Cu at (316.7, 219.1)
- added C_UVCC1: 1u, Capacitors_SMD:C_0805_HandSoldering, F.Cu at (321.5, 219.1)
- added C_VCC1: 100n, Capacitors_SMD:C_0805_HandSoldering, F.Cu at (326.2, 219.1)
- added C_VCC2: 100n, Capacitors_SMD:C_0805_HandSoldering, F.Cu at (331.0, 219.1)
- added D0,1, D0,10, D0,11, D0,12, D0,13, D0,14, D0,15, D0,16, D0,17, D0,18, D0,19, D0,2, D0,20, D0,21, D0,3, D0,4, D0,5, D0,6, D0,7, D0,8, D0,9, D1,1, D1,10, D1,11, D1,12, D1,13, D1,14, D1,15, D1,16, D1,17, D1,18, D1,19, D1,2, D1,20, D1,21, D1,3, D1,4, D1,5, D1,6, D1,7, D1,8, D1,9, D2,1, D2,10, D2,11, D2,12, D2,13, D2,14, D2,15, D2,16, D2,17, D2,18, D2,19, D2,2, D2,3, D2,4, D2,5, D2,6, D2,7, D2,8, D2,9, D3,1, D3,10, D3,11, D3,12, D3,13, D3,14, D3,15, D3,16, D3,17, D3,18, D3,19, D3,2, D3,3, D3,4, D3,5, D3,6, D3,7, D3,8, D3,9, D4,1, D4,10, D4,11, D4,12, D4,13, D4,2, D4,3, D4,4, D4,5, D4,6, D4,7, D4,8, D4,9: D, keyboard_parts:D_SOD123_axial, F.Cu at (252.4, 202.4)
- added J1: USB_C_Receptacle, Connectors_USB:USB_C_Receptacle_Amphenol_12401610E4-2A, F.Cu at (278.6, 216.7)
- added K0,1: KEYSW, keebs:Mx_Alps_100, F.Cu at (150.0, -7.14)
- added K0,10: KEYSW, keebs:Mx_Alps_100, F.Cu at (321.5, -7.14)
- added K0,11: KEYSW, keebs:Mx_Alps_100, F.Cu at (340.5, -7.14)
- added K0,12: KEYSW, keebs:Mx_Alps_100, F.Cu at (359.6, -7.14)
- added K0,13: KEYSW, keebs:Mx_Alps_100, F.Cu at (378.6, -7.14)
- added K0,14: KEYSW, keebs:Mx_Alps_100, F.Cu at (397.7, -7.14)
- added K0,15: KEYSW, keebs:Mx_Alps_100, F.Cu at (400.1, 40.5)
- added K0,16: KEYSW, keebs:Mx_Alps_100, F.Cu at (400.1, 59.5)
- added K0,17: KEYSW, keebs:Mx_Alps_100, F.Cu at (400.1, 78.6)
- added K0,18: KEYSW, keebs:Mx_Alps_200, F.Cu at (164.3, 85.7)
- added K0,19: KEYSW, keebs:Mx_Alps_100, F.Cu at (400.1, 97.6)
- added K0,2: KEYSW, keebs:Mx_Alps_100, F.Cu at (169.1, -7.14)
- added K0,20: KEYSW, keebs:Mx_Alps_100, F.Cu at (400.1, 116.7)
- added K0,21: KEYSW, keebs:Mx_Alps_100, F.Cu at (419.1, 40.5)
- added K0,3: KEYSW, keebs:Mx_Alps_100, F.Cu at (188.1, -7.14)
- added K0,4: KEYSW, keebs:Mx_Alps_100, F.Cu at (207.2, -7.14)
- added K0,5: KEYSW, keebs:Mx_Alps_100, F.Cu at (226.2, -7.14)
- added K0,6: KEYSW, keebs:Mx_Alps_100, F.Cu at (245.3, -7.14)
- added K0,7: KEYSW, keebs:Mx_Alps_100, F.Cu at (264.3, -7.14)
- added K0,8: KEYSW, keebs:Mx_Alps_100, F.Cu at (283.4, -7.14)
- added K0,9: KEYSW, keebs:Mx_Alps_100, F.Cu at (302.4, -7.14)
- added K1,1: KEYSW, keebs:Mx_Alps_100, F.Cu at (419.1, 59.5)
- added K1,10: KEYSW, keebs:Mx_Alps_100, F.Cu at (438.1, 97.6)
- added K1,11: KEYSW, keebs:Mx_Alps_100, F.Cu at (438.1, 116.7)
- added K1,12: KEYSW, keebs:Mx_Alps_100, F.Cu at (457.2, 40.5)
- added K1,13: KEYSW, keebs:Mx_Alps_100, F.Cu at (457.2, 59.5)
- added K1,14: KEYSW, keebs:Mx_Alps_100, F.Cu at (457.2, 78.6)
- added K1,15: KEYSW, keebs:Mx_Alps_100, F.Cu at (457.2, 97.6)
- added K1,16: KEYSW, keebs:Mx_Alps_100, F.Cu at (457.2, 116.7)
- added K1,17: KEYSW, keebs:Mx_Alps_100, F.Cu at (400.1, 135.7)
- added K1,18: KEYSW, keebs:Mx_Alps_150, F.Cu at (116.7, 135.7)
- added K1,19: KEYSW, keebs:Mx_Alps_100, F.Cu at (419.1, 135.7)
- added K1,2: KEYSW, keebs:Mx_Alps_100, F.Cu at (419.1, 78.6)
- added K1,20: KEYSW, keebs:Mx_Alps_100, F.Cu at (438.1, 135.7)
- added K1,21: KEYSW, keebs:Mx_Alps_100, F.Cu at (457.2, 135.7)
- added K1,3: KEYSW, keebs:Mx_Alps_100, F.Cu at (419.1, 97.6)
- added K1,4: KEYSW, keebs:Mx_Alps_200, F.Cu at (164.3, 104.8)
- added K1,5: KEYSW, keebs:Mx_Alps_150, F.Cu at (116.7, 116.7)
- added K1,6: KEYSW, keebs:Mx_Alps_100, F.Cu at (419.1, 116.7)
- added K1,7: KEYSW, keebs:Mx_Alps_100, F.Cu at (438.1, 40.5)
- added K1,8: KEYSW, keebs:Mx_Alps_100, F.Cu at (438.1, 59.5)
- added K1,9: KEYSW, keebs:Mx_Alps_100, F.Cu at (438.1, 78.6)
- added K2,1: KEYSW, keebs:Mx_Alps_100, F.Cu at (416.7, -7.14)
- added K2,10: KEYSW, keebs:Mx_Alps_100, F.Cu at (131.0, -7.14)
- added K2,11: KEYSW, keebs:Mx_Alps_100, F.Cu at (111.9, -7.14)
- added K2,12: KEYSW, keebs:Mx_Alps_100, F.Cu at (92.9, -7.14)
- added K2,13: KEYSW, keebs:Mx_Alps_100, F.Cu at (73.8, -7.14)
- added K2,14: KEYSW, keebs:Mx_Alps_100, F.Cu at (54.8, -7.14)
- added K2,15: KEYSW, keebs:Mx_Alps_100, F.Cu at (476.2, 40.5)
- added K2,16: KEYSW, keebs:Mx_Alps_225, F.Cu at (335.8, 57.1)
- added K2,17: KEYSW, keebs:Mx_Alps_100, F.Cu at (476.2, 59.5)
- added K2,18: KEYSW, keebs:Mx_Alps_100, F.Cu at (476.2, 78.6)
- added K2,19: KEYSW, keebs:Mx_Alps_100, F.Cu at (476.2, 97.6)
- added K2,2: KEYSW, keebs:Mx_Alps_100, F.Cu at (381.0, 40.5)
- added K2,3: KEYSW, keebs:Mx_Alps_100, F.Cu at (381.0, 59.5)
- added K2,4: KEYSW, keebs:Mx_Alps_175, F.Cu at (119.1, 85.7)
- added K2,5: KEYSW, keebs:Mx_Alps_100, F.Cu at (381.0, 78.6)
- added K2,6: KEYSW, keebs:Mx_Alps_100, F.Cu at (381.0, 97.6)
- added K2,7: KEYSW, keebs:Mx_Alps_100, F.Cu at (381.0, 116.7)
- added K2,8: KEYSW, keebs:Mx_Alps_100, F.Cu at (381.0, 135.7)
- added K2,9: KEYSW, keebs:Mx_Alps_100, F.Cu at (435.8, -7.14)
- added K3,1: KEYSW, keebs:Mx_Alps_100, F.Cu at (476.2, 116.7)
- added K3,10: KEYSW, keebs:Mx_Alps_100, F.Cu at (495.3, 40.5)
- added K3,11: KEYSW, keebs:Mx_Alps_100, F.Cu at (514.4, 135.7)
- added K3,12: KEYSW, keebs:Mx_Alps_100, F.Cu at (514.4, 116.7)
- added K3,13: KEYSW, keebs:Mx_Alps_100, F.Cu at (514.4, 97.6)
- added K3,14: KEYSW, keebs:Mx_Alps_100, F.Cu at (514.4, 78.6)
- added K3,15: KEYSW, keebs:Mx_Alps_100, F.Cu at (514.4, 59.5)
- added K3,16: KEYSW, keebs:Mx_Alps_275, F.Cu at (159.5, 57.1)
- added K3,17: KEYSW, keebs:Mx_Alps_100, F.Cu at (514.4, 40.5)
- added K3,18: KEYSW, keebs:Mx_Alps_100, F.Cu at (533.4, 135.7)
- added K3,19: KEYSW, keebs:Mx_Alps_100, F.Cu at (533.4, 116.7)
- added K3,2: KEYSW, keebs:Mx_Alps_100, F.Cu at (476.2, 135.7)
- added K3,3: KEYSW, keebs:Mx_Alps_100, F.Cu at (495.3, 135.7)
- added K3,4: KEYSW, keebs:Mx_Alps_200, F.Cu at (164.3, 123.8)
- added K3,5: KEYSW, keebs:Mx_Alps_225, F.Cu at (335.8, 76.2)
- added K3,6: KEYSW, keebs:Mx_Alps_100, F.Cu at (495.3, 116.7)
- added K3,7: KEYSW, keebs:Mx_Alps_100, F.Cu at (495.3, 97.6)
- added K3,8: KEYSW, keebs:Mx_Alps_100, F.Cu at (495.3, 78.6)
- added K3,9: KEYSW, keebs:Mx_Alps_100, F.Cu at (495.3, 59.5)
- added K4,1: KEYSW, keebs:Mx_Alps_200, F.Cu at (164.3, 142.9)
- added K4,10: KEYSW, keebs:Mx_Alps_125, F.Cu at (76.2, 47.6)
- added K4,11: KEYSW, keebs:Mx_Alps_100, F.Cu at (533.4, 78.6)
- added K4,12: KEYSW, keebs:Mx_Alps_100, F.Cu at (533.4, 59.5)
- added K4,13: KEYSW, keebs:Mx_Alps_100, F.Cu at (533.4, 40.5)
- added K4,2: KEYSW, keebs:Mx_Alps_100, F.Cu at (533.4, 97.6)
- added K4,3: KEYSW, keebs:Mx_Alps_125, F.Cu at (76.2, 85.7)
- added K4,4: KEYSW, keebs:Mx_Alps_125, F.Cu at (76.2, 104.8)
- added K4,5: KEYSW, keebs:Mx_Alps_125, F.Cu at (76.2, 123.8)
- added K4,6: KEYSW, keebs:Mx_Alps_625, F.Cu at (250.0, 57.1)
- added K4,7: KEYSW, keebs:Mx_Alps_125, F.Cu at (76.2, 142.9)
- added K4,8: KEYSW, keebs:Mx_Alps_125, F.Cu at (76.2, 161.9)
- added K4,9: KEYSW, keebs:Mx_Alps_125, F.Cu at (76.2, 66.7)
- added R_HWB1: 1k, Resistors_SMD:R_0805_HandSoldering, F.Cu at (252.4, 202.4)
- added R_RST1: 10k, Resistors_SMD:R_0805_HandSoldering, F.Cu at (252.4, 202.4)
- added R_USB1, R_USB2: 5.1k, Resistors_SMD:R_0805_HandSoldering, F.Cu at (252.4, 202.4)
- added R_USB3, R_USB4: 22, Resistors_SMD:R_0805_HandSoldering, F.Cu at (252.4, 202.4)
- added SW1: SW_PUSH, Buttons_Switches_SMD:SW_SPST_TL3342, F.Cu at (338.1, 207.2)
- added U1: AT90USB1286, Housings_QFP:TQFP-64_14x14mm_Pitch0.8mm, F.Cu at (359.6, 214.3)
- added Y1: 16M, Crystals:Crystal_SMD_SeikoEpson_FA238-4pin_3.2x2.5mm_HandSoldering, F.Cu at (340.5, 219.1)

Commit message: 2017.11.15 Update
- Layed out most electronics on the board
Parts:
- C_AVCC1, C_CAP1, C_CLK1, C_CLK2, C_REF1, C_UVCC1, C_VCC1, C_VCC2, D0,1, D0,10, D0,11, D0,12, D0,13, D0,14, D0,15, D0,16, D0,17, D0,18, D0,19, D0,2, D0,20, D0,21, D0,3, D0,4, D0,5, D0,6, D0,7, D0,8, D0,9, D1,1, D1,10, D1,11, D1,12, D1,13, D1,14, D1,15, D1,16, D1,17, D1,18, D1,19, D1,2, D1,20, D1,21, D1,3, D1,4, D1,5, D1,6, D1,7, D1,8, D1,9, D2,1, D2,10, D2,11, D2,12, D2,13, D2,14, D2,15, D2,16, D2,17, D2,18, D2,19, D2,2, D2,3, D2,4, D2,5, D2,6, D2,7, D2,8, D2,9, D3,1, D3,10, D3,11, D3,12, D3,13, D3,14, D3,15, D3,16, D3,17, D3,18, D3,19, D3,2, D3,3, D3,4, D3,5, D3,6, D3,7, D3,8, D3,9, D4,1, D4,10, D4,11, D4,12, D4,13, D4,2, D4,3, D4,4, D4,5, D4,6, D4,7, D4,8, D4,9, J1, R_HWB1, R_RST1, R_USB1, R_USB2, R_USB3, R_USB4, SW1, U1: moved to B.Cu
- Y1: footprint Crystals:Crystal_SMD_SeikoEpson_FA238-4pin_3.2x2.5mm_HandSoldering -> Crystals:Crystal_SMD_SeikoEpson_FA238-4pin_3.2x2.5mm; moved to B.Cu
- moved K4,2 445.5 mm to (88.1, 111.9)
- moved K3,1 426.9 mm to (50.0, 92.9)
- moved K3,2 409.4 mm to (69.1, 92.9)
- moved K3,3 409.4 mm to (88.1, 92.9)
- moved K2,1 375.5 mm to (50.0, 73.8)
- moved K1,1 369.1 mm to (50.0, 54.8)
- moved K1,2 350.9 mm to (69.1, 54.8)
- moved K1,3 333.8 mm to (88.1, 54.8)
- moved K3,6 327.1 mm to (169.1, 92.9)
- moved K4,10 320.8 mm to (390.5, 111.9)
- moved K2,2 313.7 mm to (69.1, 73.8)
- moved K3,7 307.2 mm to (188.1, 92.9)
- moved K4,9 294.0 mm to (366.7, 111.9)
- moved K2,3 293.2 mm to (88.1, 73.8)
- moved K3,8 288.5 mm to (207.2, 92.9)
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Routing:
- added copper zone on B.Cu, net GND
- added copper zone on F.Cu, net GND
Other:
- board outline added: 419.1 x 97.6 mm

Commit message: 2017.12.19 Update
Parts:
- moved J1 44.7 mm to (439.9, 29.2)
- moved C_VCC1 42.1 mm to (288.1, 107.2)
- moved C_AVCC1 37.2 mm to (288.1, 111.9)
- moved C_REF1 35.8 mm to (259.6, 109.5), turned to 180 degrees
- moved C_VCC2 35.4 mm to (288.1, 109.5)
- moved C_UVCC1 33.4 mm to (259.6, 107.2)
- moved R_RST1 24.3 mm to (259.6, 114.3), turned to 180 degrees
- moved R_USB2 20.0 mm to (396.5, 50.0), turned to 90 degrees
- moved R_USB1 12.4 mm to (398.9, 50.0), turned to 270 degrees
- moved SW1 4.76 mm to (285.8, 119.1)
- moved C_CLK2 2.38 mm to (266.7, 119.1)
- moved U1 2.38 mm to (273.8, 109.5)
- moved R_HWB1 2.38 mm to (259.6, 111.9)
- moved C_CAP1 2.38 mm to (288.1, 114.3)
- moved Y1 1.79 mm to (262.5, 119.1)
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Other:
- board size 419.1 x 97.6 mm -> 419.1 x 99.4 mm

Commit message: 2018.01.22 Update
- Most of the routing done for the new setup
Parts:
- moved R_RST1 20.7 mm to (279.2, 120.8), turned to 270 degrees
- moved C_CLK1 3.99 mm to (261.9, 120.8)
- moved Y1 3.47 mm to (265.5, 120.8)
- moved C_CLK2 2.98 mm to (269.1, 120.8)
- moved C_AVCC1 2.38 mm to (290.5, 111.9)
- moved C_CAP1 2.38 mm to (290.5, 114.3)
- moved C_VCC1 2.38 mm to (290.5, 107.2)
- moved C_VCC2 2.38 mm to (290.5, 109.5)
- moved C_REF1 2.38 mm to (257.2, 109.5)
- moved C_UVCC1 2.38 mm to (257.2, 107.2)
- moved R_HWB1 2.38 mm to (257.2, 111.9)
- moved SW1 1.28 mm to (285.2, 120.2)
Routing:
- net /col00: track 0.00 -> 319.0 mm, vias 0 -> 1
- net /col01: track 0.00 -> 295.3 mm, vias 0 -> 1
- net /col02: track 0.00 -> 282.0 mm, vias 0 -> 1
- net /col20: track 0.00 -> 270.5 mm, vias 0 -> 1
- net /col19: track 0.00 -> 252.4 mm, vias 0 -> 1
- net /col03: track 0.00 -> 252.4 mm, vias 0 -> 1
- net /col04: track 0.00 -> 247.3 mm, vias 0 -> 1
- net /col18: track 0.00 -> 233.9 mm, vias 0 -> 1
- net /col05: track 0.00 -> 215.6 mm, vias 0 -> 1
- net /col17: track 0.00 -> 210.9 mm, vias 0 -> 1
- net /row4: track 0.00 -> 198.4 mm
- net /col06: track 0.00 -> 194.1 mm, vias 0 -> 1
- net /col16: track 0.00 -> 192.4 mm, vias 0 -> 1
- net /col15: track 0.00 -> 178.7 mm, vias 0 -> 1
- net /col14: track 0.00 -> 172.3 mm, vias 0 -> 1
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
Commit message: 2018.01.24 Update
- Almost all routing complete
- Only Vcc lines remain to connect
Parts:
- moved R_USB3 2.38 mm to (401.2, 50.0)
- moved R_USB4 2.38 mm to (403.6, 50.0)
- moved C_AVCC1 1.19 mm to (291.7, 111.9)
- moved C_CAP1 1.19 mm to (291.7, 114.3)
- moved C_VCC1 1.19 mm to (291.7, 107.2)
- moved C_VCC2 1.19 mm to (291.7, 109.5)
- turned C_UVCC1 to 180 degrees
- turned R_USB2 to 270 degrees
Routing:
- net /row0: track 0.00 -> 508.5 mm, vias 0 -> 1
- net /row1: track 0.00 -> 487.7 mm, vias 0 -> 1
- net /row2: track 0.00 -> 463.4 mm, vias 0 -> 1
- net /row3: track 0.00 -> 438.7 mm, vias 0 -> 5
- net /row4: track 198.4 -> 430.9 mm, vias 0 -> 3
- net Net-(R_USB4-Pad1): track 0.00 -> 193.1 mm, vias 0 -> 2
- net Net-(R_USB3-Pad1): track 0.00 -> 188.1 mm, vias 0 -> 2
- net Net-(J1-PadA7): track 6.68 -> 67.3 mm
- net Net-(J1-PadB5): track 0.00 -> 60.6 mm, vias 0 -> 2
- net Net-(J1-PadA5): track 0.00 -> 56.2 mm
- net Net-(J1-PadA6): track 1.80 -> 57.6 mm, vias 0 -> 2
- net Net-(C_REF1-Pad1): track 0.00 -> 25.1 mm, vias 0 -> 2
- net Net-(R_HWB1-Pad2): track 0.00 -> 19.8 mm, vias 0 -> 2
- net Net-(C_CAP1-Pad1): track 0.00 -> 12.9 mm
- net /col09: track 135.6 -> 137.1 mm
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
Commit message: 2018.01.24 Update 2
- Vcc line now routed
- Further cleanup is needed
Parts:
- moved C_VCC1 34.9 mm to (257.2, 111.9), turned to 180 degrees
- moved C_UVCC1 31.3 mm to (288.1, 111.9), turned to 0 degrees
- moved C_CAP1 6.58 mm to (291.1, 120.8), turned to 270 degrees
- moved C_AVCC1 4.29 mm to (288.1, 109.5)
- moved C_VCC2 4.29 mm to (288.1, 107.2)
- moved R_HWB1 2.38 mm to (257.2, 109.5)
- moved C_REF1 2.38 mm to (257.2, 107.2)
Routing:
- net VCC: track 3.61 -> 352.6 mm, vias 0 -> 4
- net Net-(C_CAP1-Pad1): track 12.9 -> 31.1 mm, vias 0 -> 2
- net Net-(R_USB4-Pad1): track 193.1 -> 198.0 mm
- net Net-(R_USB3-Pad1): track 188.1 -> 192.8 mm
- net Net-(R_HWB1-Pad2): track 19.8 -> 16.8 mm, vias 2 -> 0
- net Net-(C_REF1-Pad1): track 25.1 -> 27.9 mm
- net /col00: track 319.0 -> 317.7 mm
- net Net-(J1-PadB5): track 60.6 -> 60.0 mm
- net Net-(R_RST1-Pad1): track 21.5 -> 20.9 mm
- net /row3: vias 5 -> 4

Commit message: 2018.01.25 Update
- Routing should be complete
- Did more cleanup, GND lines/pins connected
Parts:
- moved R_USB3 2.38 mm to (403.6, 50.0)
- moved R_USB4 2.38 mm to (401.2, 50.0)
Routing:
- net GND: track 9.12 -> 430.8 mm, vias 0 -> 12
- net VCC: track 352.6 -> 336.4 mm, vias 4 -> 6
- net Net-(J1-PadA7): track 67.3 -> 55.6 mm
- net /col05: track 215.6 -> 221.0 mm
- net Net-(R_USB4-Pad1): track 198.0 -> 192.9 mm
- net Net-(J1-PadA6): track 57.6 -> 52.8 mm, vias 2 -> 0
- net Net-(J1-PadA5): track 56.2 -> 52.4 mm
- net Net-(R_USB3-Pad1): track 192.8 -> 194.8 mm
- net /col15: track 178.7 -> 176.7 mm
- net Net-(J1-PadB5): track 60.0 -> 61.7 mm
- net /row4: track 430.7 -> 432.2 mm
- net /row3: vias 4 -> 3
- net /col17: vias 1 -> 2

Commit message: 2018.03.15 Update
- Updated labels on switches and diodes to better match array subscripts
- Started preliminary C code for the firmware
Parts:
- renumbered D0,1 to D0,0, D0,2 to D0,1, D0,11 to D0,10, D0,12 to D0,11, D0,13 to D0,12, D0,14 to D0,13, D0,15 to D0,14, D0,16 to D0,15, D0,17 to D0,16, D0,18 to D0,17, D0,19 to D0,18, D0,20 to D0,19, D0,3 to D0,2, D0,21 to D0,20, D0,4 to D0,3, D0,5 to D0,4, D0,6 to D0,5, D0,7 to D0,6, D0,8 to D0,7, D0,9 to D0,8, D0,10 to D0,9, D1,1 to D1,0, D1,2 to D1,1, D1,11 to D1,10, D1,12 to D1,11, D1,13 to D1,12, D1,14 to D1,13, D1,15 to D1,14, D1,16 to D1,15, D1,17 to D1,16, D1,18 to D1,17, D1,19 to D1,18, D1,20 to D1,19, D1,3 to D1,2, D1,21 to D1,20, D1,4 to D1,3, D1,5 to D1,4, D1,6 to D1,5, D1,7 to D1,6, D1,8 to D1,7, D1,9 to D1,8, D1,10 to D1,9, D2,1 to D2,0, D2,2 to D2,1, D2,16 to D2,17, D2,17 to D2,18, D2,18 to D2,19, D2,3 to D2,2, D2,19 to D2,20, D3,1 to D3,0, D3,2 to D3,1, D3,11 to D3,10, D3,12 to D3,11, D3,13 to D3,12, D3,14 to D3,13, D3,15 to D3,14, D3,17 to D3,18, D3,18 to D3,19, D3,3 to D3,2, D3,19 to D3,20, D3,4 to D3,3, D3,5 to D3,4, D3,6 to D3,5, D3,7 to D3,6, D3,8 to D3,7, D3,9 to D3,8, D3,10 to D3,9, D4,1 to D4,0, D4,7 to D4,13, D4,8 to D4,14, D4,9 to D4,16, D4,10 to D4,17, D4,11 to D4,18, D4,12 to D4,19, D4,13 to D4,20, D4,3 to D4,4, D4,4 to D4,5, D4,5 to D4,6, D4,6 to D4,9, K0,1 to K0,0, K0,2 to K0,1, K0,11 to K0,10, K0,12 to K0,11, K0,13 to K0,12, K0,14 to K0,13, K0,15 to K0,14, K0,16 to K0,15, K0,17 to K0,16, K0,18 to K0,17, K0,19 to K0,18, K0,20 to K0,19, K0,3 to K0,2, K0,21 to K0,20, K0,4 to K0,3, K0,5 to K0,4, K0,6 to K0,5, K0,7 to K0,6, K0,8 to K0,7, K0,9 to K0,8, K0,10 to K0,9, K1,1 to K1,0, K1,2 to K1,1, K1,11 to K1,10, K1,12 to K1,11, K1,13 to K1,12, K1,14 to K1,13, K1,15 to K1,14, K1,16 to K1,15, K1,17 to K1,16, K1,18 to K1,17, K1,19 to K1,18, K1,20 to K1,19, K1,3 to K1,2, K1,21 to K1,20, K1,4 to K1,3, K1,5 to K1,4, K1,6 to K1,5, K1,7 to K1,6, K1,8 to K1,7, K1,9 to K1,8, K1,10 to K1,9, K2,1 to K2,0, K2,2 to K2,1, K2,16 to K2,17, K2,17 to K2,18, K2,18 to K2,19, K2,3 to K2,2, K2,19 to K2,20, K3,1 to K3,0, K3,2 to K3,1, K3,11 to K3,10, K3,12 to K3,11, K3,13 to K3,12, K3,14 to K3,13, K3,15 to K3,14, K3,17 to K3,18, K3,18 to K3,19, K3,3 to K3,2, K3,19 to K3,20, K3,4 to K3,3, K3,5 to K3,4, K3,6 to K3,5, K3,7 to K3,6, K3,8 to K3,7, K3,9 to K3,8, K3,10 to K3,9, K4,1 to K4,0, K4,7 to K4,13, K4,8 to K4,14, K4,9 to K4,16, K4,10 to K4,17, K4,11 to K4,18, K4,12 to K4,19, K4,13 to K4,20, K4,3 to K4,4, K4,4 to K4,5, K4,5 to K4,6, K4,6 to K4,9
