File: PCB/JayKey1.kicad_pcb (KiCad board)
At the start: 2 copper layers, 419.1 x 101.2 mm, 212 parts, among them J1 USB_C_Receptacle_USB2.0, J2 USB_C_Receptacle_USB2.0, K0,0 KEYSW, K0,1 KEYSW, K0,10 KEYSW, K0,11 KEYSW, K0,12 KEYSW, K0,13 KEYSW, K0,14 KEYSW, K0,15 KEYSW, K0,16 KEYSW, K0,17 KEYSW, K0,18 KEYSW, K0,19 KEYSW, K0,2 KEYSW, K0,20 KEYSW, K0,3 KEYSW, K0,4 KEYSW, K0,5 KEYSW, K0,6 KEYSW, K0,7 KEYSW, K0,8 KEYSW, K0,9 KEYSW, K1,0 KEYSW, K1,1 KEYSW, K1,10 KEYSW, K1,11 KEYSW, K1,12 KEYSW, K1,13 KEYSW, K1,14 KEYSW, K1,15 KEYSW, K1,16 KEYSW, K1,17 KEYSW, K1,18 KEYSW, K1,19 KEYSW, K1,2 KEYSW, K1,20 KEYSW, K1,3 KEYSW, K1,4 KEYSW, K1,5 KEYSW, K1,6 KEYSW, K1,7 KEYSW, K1,8 KEYSW, K1,9 KEYSW, K2,0 KEYSW, K2,1 KEYSW, K2,10 KEYSW, K2,11 KEYSW, K2,12 KEYSW, K2,13 KEYSW, K2,14 KEYSW, K2,15 KEYSW, K2,17 KEYSW, K2,18 KEYSW, K2,19 KEYSW, K2,2 KEYSW, K2,20 KEYSW, K2,4 KEYSW, K2,5 KEYSW, K2,6 KEYSW, K2,7 KEYSW, K2,8 KEYSW, K2,9 KEYSW, K3,0 KEYSW, K3,1 KEYSW, K3,10 KEYSW, K3,11 KEYSW, K3,12 KEYSW, K3,13 KEYSW, K3,14 KEYSW, K3,16 KEYSW, K3,18 KEYSW, K3,19 KEYSW, K3,2 KEYSW, K3,20 KEYSW, K3,3 KEYSW, K3,4 KEYSW, K3,5 KEYSW, K3,6 KEYSW, K3,7 KEYSW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

Commit message: 2018.12.04 Nightly
Parts:
- removed D_ESD2: PESD5V0L2BT, Package_TO_SOT_SMD:SOT-23_Handsoldering
- removed D_VBUS2: D, keyboard_parts:D_SOD123_axial
- removed J2: USB_C_Receptacle_USB2.0, Connector_USB:USB_C_Receptacle_Amphenol_12401610E4-2A
- removed R_USB5, R_USB6: 5.1k, Resistors_SMD:R_0805_HandSoldering
- C_AREF1, C_AVCC1, C_CLK1, C_CLK2, C_UCAP1, C_UVCC1, C_VBUS1, C_VCC1, C_VCC2: footprint Capacitors_SMD:C_0805_HandSoldering -> Capacitor_SMD:C_0805_2012Metric_Pad1.15x1.40mm_HandSolder
- R_HWB1, R_RST1, R_USB1, R_USB2, R_USB3, R_USB4: footprint Resistors_SMD:R_0805_HandSoldering -> Resistor_SMD:R_0805_2012Metric_Pad1.15x1.40mm_HandSolder
- moved R_HWB1 26.1 mm to (255.0, 133.9)
- moved R_USB1 21.9 mm to (285.9, 116.1), turned to 0 degrees
- moved C_VCC1 20.2 mm to (273.1, 126.2)
- moved R_USB2 18.7 mm to (285.9, 118.5), turned to 0 degrees
- moved R_RST1 15.0 mm to (291.3, 111.9), turned to 0 degrees
- moved C_VCC2 14.9 mm to (273.8, 100.0), turned to 180 degrees
- moved C_VBUS1 12.9 mm to (281.2, 120.8), turned to 0 degrees
- moved C_CLK2 11.1 mm to (255.0, 129.2), turned to 0 degrees
- moved C_CLK1 10.3 mm to (268.1, 128.6), turned to 0 degrees
- moved SW1 7.17 mm to (291.7, 117.3), turned to 90 degrees
- moved C_UCAP1 5.19 mm to (285.9, 120.8), turned to 0 degrees
- moved D_VBUS1 4.53 mm to (441.7, 47.9)
- moved C_AVCC1 3.47 mm to (285.7, 107.8)
- moved C_AREF1 3.47 mm to (285.7, 105.4)
- moved U1 2.38 mm to (273.8, 111.9)
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Connections:
- net /DMINUS renamed /D_N
- net /DPLUS renamed /D_P
- net Net-(C_CLK1-Pad1) renamed /CLK_P
- net Net-(C_CLK2-Pad1) renamed /CLK_N
- net Net-(R_USB1-Pad1) renamed /D_-
- net Net-(R_USB2-Pad1) renamed /D_+
- D0,0 pad 1: /Key Matrix/row0 -> /row0
- D0,1 pad 1: /Key Matrix/row0 -> /row0
- D0,10 pad 1: /Key Matrix/row0 -> /row0
- D0,11 pad 1: /Key Matrix/row0 -> /row0
- D0,12 pad 1: /Key Matrix/row0 -> /row0
- D0,13 pad 1: /Key Matrix/row0 -> /row0
- D0,14 pad 1: /Key Matrix/row0 -> /row0
- D0,15 pad 1: /Key Matrix/row0 -> /row0
- D0,16 pad 1: /Key Matrix/row0 -> /row0
- D0,17 pad 1: /Key Matrix/row0 -> /row0
- D0,18 pad 1: /Key Matrix/row0 -> /row0
- D0,19 pad 1: /Key Matrix/row0 -> /row0
- D0,2 pad 1: /Key Matrix/row0 -> /row0
- D0,20 pad 1: /Key Matrix/row0 -> /row0
- D0,3 pad 1: /Key Matrix/row0 -> /row0
- D0,4 pad 1: /Key Matrix/row0 -> /row0
- D0,5 pad 1: /Key Matrix/row0 -> /row0
- D0,6 pad 1: /Key Matrix/row0 -> /row0
- D0,7 pad 1: /Key Matrix/row0 -> /row0
- D0,8 pad 1: /Key Matrix/row0 -> /row0
- D0,9 pad 1: /Key Matrix/row0 -> /row0
- D1,0 pad 1: /Key Matrix/row1 -> /row1
- D1,1 pad 1: /Key Matrix/row1 -> /row1
- D1,10 pad 1: /Key Matrix/row1 -> /row1
- D1,11 pad 1: /Key Matrix/row1 -> /row1
- D1,12 pad 1: /Key Matrix/row1 -> /row1
- D1,13 pad 1: /Key Matrix/row1 -> /row1
- D1,14 pad 1: /Key Matrix/row1 -> /row1
- D1,15 pad 1: /Key Matrix/row1 -> /row1
- D1,16 pad 1: /Key Matrix/row1 -> /row1
- D1,17 pad 1: /Key Matrix/row1 -> /row1
- D1,18 pad 1: /Key Matrix/row1 -> /row1
- D1,19 pad 1: /Key Matrix/row1 -> /row1
- D1,2 pad 1: /Key Matrix/row1 -> /row1
- D1,20 pad 1: /Key Matrix/row1 -> /row1
- D1,3 pad 1: /Key Matrix/row1 -> /row1
- D1,4 pad 1: /Key Matrix/row1 -> /row1
- D1,5 pad 1: /Key Matrix/row1 -> /row1
- D1,6 pad 1: /Key Matrix/row1 -> /row1
- D1,7 pad 1: /Key Matrix/row1 -> /row1
- D1,8 pad 1: /Key Matrix/row1 -> /row1
- D1,9 pad 1: /Key Matrix/row1 -> /row1
- D2,0 pad 1: /Key Matrix/row2 -> /row2
- D2,1 pad 1: /Key Matrix/row2 -> /row2
- D2,10 pad 1: /Key Matrix/row2 -> /row2
- D2,11 pad 1: /Key Matrix/row2 -> /row2
- D2,12 pad 1: /Key Matrix/row2 -> /row2
- D2,13 pad 1: /Key Matrix/row2 -> /row2
- D2,14 pad 1: /Key Matrix/row2 -> /row2
- D2,15 pad 1: /Key Matrix/row2 -> /row2
- D2,17 pad 1: /Key Matrix/row2 -> /row2
- D2,18 pad 1: /Key Matrix/row2 -> /row2
- D2,19 pad 1: /Key Matrix/row2 -> /row2
- D2,2 pad 1: /Key Matrix/row2 -> /row2
- D2,20 pad 1: /Key Matrix/row2 -> /row2
- D2,4 pad 1: /Key Matrix/row2 -> /row2
- D2,5 pad 1: /Key Matrix/row2 -> /row2
- D2,6 pad 1: /Key Matrix/row2 -> /row2
- D2,7 pad 1: /Key Matrix/row2 -> /row2
- D2,8 pad 1: /Key Matrix/row2 -> /row2
- D2,9 pad 1: /Key Matrix/row2 -> /row2
- D3,0 pad 1: /Key Matrix/row3 -> /row3
- D3,1 pad 1: /Key Matrix/row3 -> /row3
- D3,10 pad 1: /Key Matrix/row3 -> /row3
- D3,11 pad 1: /Key Matrix/row3 -> /row3
- D3,12 pad 1: /Key Matrix/row3 -> /row3
- D3,13 pad 1: /Key Matrix/row3 -> /row3
- D3,14 pad 1: /Key Matrix/row3 -> /row3
- D3,16 pad 1: /Key Matrix/row3 -> /row3
- D3,18 pad 1: /Key Matrix/row3 -> /row3
- D3,19 pad 1: /Key Matrix/row3 -> /row3
- D3,2 pad 1: /Key Matrix/row3 -> /row3
- D3,20 pad 1: /Key Matrix/row3 -> /row3
- D3,3 pad 1: /Key Matrix/row3 -> /row3
- D3,4 pad 1: /Key Matrix/row3 -> /row3
- D3,5 pad 1: /Key Matrix/row3 -> /row3
- D3,6 pad 1: /Key Matrix/row3 -> /row3
- D3,7 pad 1: /Key Matrix/row3 -> /row3
- D3,8 pad 1: /Key Matrix/row3 -> /row3
- D3,9 pad 1: /Key Matrix/row3 -> /row3
- D4,0 pad 1: /Key Matrix/row4 -> /row4
- D4,13 pad 1: /Key Matrix/row4 -> /row4
- D4,14 pad 1: /Key Matrix/row4 -> /row4
- D4,16 pad 1: /Key Matrix/row4 -> /row4
- D4,17 pad 1: /Key Matrix/row4 -> /row4
- D4,18 pad 1: /Key Matrix/row4 -> /row4
- D4,19 pad 1: /Key Matrix/row4 -> /row4
- D4,2 pad 1: /Key Matrix/row4 -> /row4
- D4,20 pad 1: /Key Matrix/row4 -> /row4
- D4,4 pad 1: /Key Matrix/row4 -> /row4
- D4,5 pad 1: /Key Matrix/row4 -> /row4
- D4,6 pad 1: /Key Matrix/row4 -> /row4
- D4,9 pad 1: /Key Matrix/row4 -> /row4
- J1 pad A8: Net-(J1-PadA8) -> (no net)
- J1 pad B8: Net-(J1-PadB8) -> (no net)
- K0,0 pad 1: /Key Matrix/col00 -> /col00
- K0,1 pad 1: /Key Matrix/col01 -> /col01
- K0,10 pad 1: /Key Matrix/col10 -> /col10
- K0,11 pad 1: /Key Matrix/col11 -> /col11
- K0,12 pad 1: /Key Matrix/col12 -> /col12
- K0,13 pad 1: /Key Matrix/col13 -> /col13
- K0,14 pad 1: /Key Matrix/col14 -> /col14
- K0,15 pad 1: /Key Matrix/col15 -> /col15
- K0,16 pad 1: /Key Matrix/col16 -> /col16
- K0,17 pad 1: /Key Matrix/col17 -> /col17
- K0,18 pad 1: /Key Matrix/col18 -> /col18
- K0,19 pad 1: /Key Matrix/col19 -> /col19
- K0,2 pad 1: /Key Matrix/col02 -> /col02
- K0,20 pad 1: /Key Matrix/col20 -> /col20
- K0,3 pad 1: /Key Matrix/col03 -> /col03
- K0,4 pad 1: /Key Matrix/col04 -> /col04
- K0,5 pad 1: /Key Matrix/col05 -> /col05
- K0,6 pad 1: /Key Matrix/col06 -> /col06
- K0,7 pad 1: /Key Matrix/col07 -> /col07
- K0,8 pad 1: /Key Matrix/col08 -> /col08
- K0,9 pad 1: /Key Matrix/col09 -> /col09
- K1,0 pad 1: /Key Matrix/col00 -> /col00
- K1,1 pad 1: /Key Matrix/col01 -> /col01
- K1,10 pad 1: /Key Matrix/col10 -> /col10
- K1,11 pad 1: /Key Matrix/col11 -> /col11
- K1,12 pad 1: /Key Matrix/col12 -> /col12
- K1,13 pad 1: /Key Matrix/col13 -> /col13
- K1,14 pad 1: /Key Matrix/col14 -> /col14
- K1,15 pad 1: /Key Matrix/col15 -> /col15
- K1,16 pad 1: /Key Matrix/col16 -> /col16
- K1,17 pad 1: /Key Matrix/col17 -> /col17
- K1,18 pad 1: /Key Matrix/col18 -> /col18
- K1,19 pad 1: /Key Matrix/col19 -> /col19
- K1,2 pad 1: /Key Matrix/col02 -> /col02
- K1,20 pad 1: /Key Matrix/col20 -> /col20
- K1,3 pad 1: /Key Matrix/col03 -> /col03
- K1,4 pad 1: /Key Matrix/col04 -> /col04
- K1,5 pad 1: /Key Matrix/col05 -> /col05
- K1,6 pad 1: /Key Matrix/col06 -> /col06
- K1,7 pad 1: /Key Matrix/col07 -> /col07
- K1,8 pad 1: /Key Matrix/col08 -> /col08
- K1,9 pad 1: /Key Matrix/col09 -> /col09
- K2,0 pad 1: /Key Matrix/col00 -> /col00
- K2,1 pad 1: /Key Matrix/col01 -> /col01
- K2,10 pad 1: /Key Matrix/col10 -> /col10
- K2,11 pad 1: /Key Matrix/col11 -> /col11
- K2,12 pad 1: /Key Matrix/col12 -> /col12
- K2,13 pad 1: /Key Matrix/col13 -> /col13
- K2,14 pad 1: /Key Matrix/col14 -> /col14
- K2,15 pad 1: /Key Matrix/col15 -> /col15
- K2,17 pad 1: /Key Matrix/col17 -> /col17
- K2,18 pad 1: /Key Matrix/col18 -> /col18
- K2,19 pad 1: /Key Matrix/col19 -> /col19
- K2,2 pad 1: /Key Matrix/col02 -> /col02
- K2,20 pad 1: /Key Matrix/col20 -> /col20
- K2,4 pad 1: /Key Matrix/col04 -> /col04
- K2,5 pad 1: /Key Matrix/col05 -> /col05
- K2,6 pad 1: /Key Matrix/col06 -> /col06
- K2,7 pad 1: /Key Matrix/col07 -> /col07
- K2,8 pad 1: /Key Matrix/col08 -> /col08
- K2,9 pad 1: /Key Matrix/col09 -> /col09
- K3,0 pad 1: /Key Matrix/col00 -> /col00
- K3,1 pad 1: /Key Matrix/col01 -> /col01
- K3,10 pad 1: /Key Matrix/col10 -> /col10
- K3,11 pad 1: /Key Matrix/col11 -> /col11
- K3,12 pad 1: /Key Matrix/col12 -> /col12
- K3,13 pad 1: /Key Matrix/col13 -> /col13
- K3,14 pad 1: /Key Matrix/col14 -> /col14
- K3,16 pad 1: /Key Matrix/col16 -> /col16
- K3,18 pad 1: /Key Matrix/col18 -> /col18
- K3,19 pad 1: /Key Matrix/col19 -> /col19
- K3,2 pad 1: /Key Matrix/col02 -> /col02
- K3,20 pad 1: /Key Matrix/col20 -> /col20
- K3,3 pad 1: /Key Matrix/col03 -> /col03
- K3,4 pad 1: /Key Matrix/col04 -> /col04
- K3,5 pad 1: /Key Matrix/col05 -> /col05
- K3,6 pad 1: /Key Matrix/col06 -> /col06
- K3,7 pad 1: /Key Matrix/col07 -> /col07
- K3,8 pad 1: /Key Matrix/col08 -> /col08
- K3,9 pad 1: /Key Matrix/col09 -> /col09
- K4,0 pad 1: /Key Matrix/col00 -> /col00
- K4,13 pad 1: /Key Matrix/col13 -> /col13
- K4,14 pad 1: /Key Matrix/col14 -> /col14
- K4,16 pad 1: /Key Matrix/col16 -> /col16
- K4,17 pad 1: /Key Matrix/col17 -> /col17
- K4,18 pad 1: /Key Matrix/col18 -> /col18
- K4,19 pad 1: /Key Matrix/col19 -> /col19
- K4,2 pad 1: /Key Matrix/col02 -> /col02
- K4,20 pad 1: /Key Matrix/col20 -> /col20
- K4,4 pad 1: /Key Matrix/col04 -> /col04
- K4,5 pad 1: /Key Matrix/col05 -> /col05
- K4,6 pad 1: /Key Matrix/col06 -> /col06
- K4,9 pad 1: /Key Matrix/col09 -> /col09
- U1 pad 1: Net-(U1-Pad1) -> (no net)
- U1 pad 10: Net-(U1-Pad10) -> (no net)
- U1 pad 11: Net-(U1-Pad11) -> (no net)
- U1 pad 12: Net-(U1-Pad12) -> (no net)
- U1 pad 13: Net-(U1-Pad13) -> (no net)
- U1 pad 14: Net-(U1-Pad14) -> (no net)
- U1 pad 15: Net-(U1-Pad15) -> (no net)
- U1 pad 16: Net-(U1-Pad16) -> (no net)
- U1 pad 17: Net-(U1-Pad17) -> (no net)
- U1 pad 18: Net-(U1-Pad18) -> (no net)
- U1 pad 19: Net-(U1-Pad19) -> (no net)
- U1 pad 2: Net-(U1-Pad2) -> (no net)
- U1 pad 25: Net-(U1-Pad25) -> (no net)
- U1 pad 26: Net-(U1-Pad26) -> (no net)
- U1 pad 27: Net-(U1-Pad27) -> (no net)
- U1 pad 33: Net-(U1-Pad33) -> (no net)
- U1 pad 34: Net-(U1-Pad34) -> (no net)
- U1 pad 49: Net-(U1-Pad49) -> (no net)
- U1 pad 50: Net-(U1-Pad50) -> (no net)
- U1 pad 51: Net-(U1-Pad51) -> (no net)
- U1 pad 9: Net-(U1-Pad9) -> (no net)
Routing:
- net /Key Matrix/row0: track 503.3 -> 0.00 mm, vias 2 -> 0
- net /Key Matrix/row1: track 486.0 -> 0.00 mm, vias 1 -> 0
- net /Key Matrix/row2: track 461.7 -> 0.00 mm, vias 1 -> 0
- net /Key Matrix/row3: track 436.3 -> 0.00 mm, vias 1 -> 0
- net /Key Matrix/row4: track 430.3 -> 0.00 mm, vias 2 -> 0
- net /Key Matrix/col00: track 309.9 -> 0.00 mm, vias 1 -> 0
- net /col00: track 0.00 -> 300.0 mm
- net /Key Matrix/col01: track 292.4 -> 0.00 mm, vias 1 -> 0
- net /Key Matrix/col02: track 280.6 -> 0.00 mm, vias 1 -> 0
- net /col01: track 0.00 -> 275.8 mm
- net /col02: track 0.00 -> 270.6 mm
- net /Key Matrix/col20: track 265.2 -> 0.00 mm, vias 1 -> 0
- net /Key Matrix/col03: track 248.4 -> 0.00 mm, vias 1 -> 0
- net /Key Matrix/col19: track 246.1 -> 0.00 mm, vias 1 -> 0
- net /Key Matrix/col04: track 245.8 -> 0.00 mm, vias 1 -> 0
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- removed copper zone on F.Cu, net GND
Other:
- net class USB added: clearance 0.2, trace_width 0.2, via_dia 0.6, via_drill 0.4
- board text added: "JayKey1 by Josue Galeas (Version 2.0) Open-source and powered by TMK https://github.com/josuegaleas/JayKey1"
- board text removed: "JayKey1 by Josue Galeas (Version 1.2) https://github.com/josuegaleas/JayKey1"

Commit message: 2018.12.06 Nightly
Parts:
- moved R_HWB1 23.0 mm to (261.5, 111.9)
- moved C_CLK2 7.89 mm to (257.2, 121.6), turned to 270 degrees
- moved SW1 7.62 mm to (297.7, 112.5), turned to 0 degrees
- moved C_CLK1 7.43 mm to (265.5, 121.6), turned to 90 degrees
- moved Y1 6.05 mm to (261.3, 121.4)
- moved C_VCC1 5.49 mm to (268.9, 122.6)
- moved R_RST1 1.36 mm to (289.9, 111.9), turned to 90 degrees
Routing:
- net /col05: track 0.00 -> 215.2 mm
- net /col06: track 0.00 -> 194.8 mm
- net /col16: track 5.79 -> 196.0 mm
- net /col04: track 89.9 -> 250.3 mm
- net /col14: track 5.83 -> 165.3 mm
- net /col07: track 0.00 -> 152.4 mm
- net /col17: track 5.77 -> 157.8 mm
- net /col15: track 5.81 -> 151.6 mm
- net /col13: track 5.84 -> 144.8 mm
- net GND: track 273.3 -> 410.8 mm, vias 3 -> 6
- net /col09: track 0.00 -> 137.1 mm
- net /col08: track 0.00 -> 133.6 mm
- net /col12: track 0.00 -> 116.1 mm
- net /col18: track 5.76 -> 107.8 mm
- net /col11: track 0.00 -> 97.9 mm
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
Commit message: 2018.12.14 Nightly
Parts:
- moved R_HWB1 0.17 mm to (261.3, 111.9), turned to 90 degrees
Routing:
- net /col20: track 85.4 -> 256.4 mm, vias 0 -> 1
- net /col19: track 86.0 -> 244.8 mm
- net /col18: track 107.8 -> 234.0 mm
- net /col17: track 157.8 -> 233.1 mm
- net Net-(D3,3-Pad2): track 0.00 -> 10.1 mm
- net Net-(D0,3-Pad2): track 0.00 -> 10.1 mm
- net Net-(D4,2-Pad2): track 0.00 -> 10.1 mm
- net Net-(D4,0-Pad2): track 0.00 -> 10.1 mm
- net Net-(D1,3-Pad2): track 0.00 -> 10.1 mm
- net Net-(D1,0-Pad2): track 0.00 -> 10.1 mm
- net Net-(D0,0-Pad2): track 0.00 -> 10.1 mm
- net Net-(D3,0-Pad2): track 0.00 -> 10.1 mm
- net Net-(D2,0-Pad2): track 0.00 -> 10.1 mm
- net Net-(D1,2-Pad2): track 0.00 -> 10.1 mm
- net Net-(D1,1-Pad2): track 0.00 -> 10.1 mm
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
Commit message: 2018.12.14 Nightly 2
Connections:
- C_AVCC1 pad 1: VBUS -> VCC
- C_UVCC1 pad 1: VBUS -> VCC
- C_VBUS1 pad 1: VBUS -> VCC
- C_VCC1 pad 1: VBUS -> VCC
- C_VCC2 pad 1: VBUS -> VCC
- D_VBUS1 pad 1: VBUS -> VCC
- R_RST1 pad 2: VBUS -> VCC
- U1 pad 21: VBUS -> VCC
- U1 pad 3: VBUS -> VCC
- U1 pad 52: VBUS -> VCC
- U1 pad 64: VBUS -> VCC
- U1 pad 8: VBUS -> VCC
Routing:
- net /row1: track 3.06 -> 490.8 mm
- net /row0: track 24.2 -> 508.8 mm
- net /row2: track 3.08 -> 474.1 mm
- net /row3: track 3.09 -> 447.5 mm, vias 1 -> 7
- net /row4: track 77.3 -> 436.5 mm
- net VCC: track 0.00 -> 296.4 mm
- net VBUS: track 317.8 -> 21.4 mm
- net /col17: track 233.1 -> 203.4 mm, vias 0 -> 1
- net Net-(D4,9-Pad2): track 0.00 -> 10.1 mm
- net Net-(D4,6-Pad2): track 0.00 -> 10.1 mm
- net Net-(D4,5-Pad2): track 0.00 -> 10.1 mm
- net Net-(D4,4-Pad2): track 0.00 -> 10.1 mm
- net Net-(D1,8-Pad2): track 0.00 -> 10.1 mm
- net Net-(D0,6-Pad2): track 0.00 -> 10.1 mm
- net Net-(D3,6-Pad2): track 0.00 -> 10.1 mm
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