File: PCB/JayKey1.sch (KiCad schematic (older format))
At the start: 0 parts

Commit message: 2017.11.14 Nightly
Parts:
- added C_AVCC, C_REF, C_VCC1, C_VCC2: 100n, symbol C
- added C_CAP, C_UVCC: 1u, symbol C
- added C_CLK1, C_CLK2: 22p, symbol C
- added J1: USB_C_Receptacle, symbol USB_C_Receptacle
- added R_HWB: 1k, symbol R
- added R_RST: 10k, symbol R
- added R_USB1, R_USB2: 5.1k, symbol R
- added R_USB3, R_USB4: 22, symbol R
- added SW1: SW_PUSH, symbol SW_PUSH
- added U1: AT90USB1286, symbol AT90USB1286
- added Y1: 16M, symbol Crystal_GND23
Connections:
- new net: R_RST.1, SW1.2, U1.20 (~RESET)
- new net: C_CLK2.1, U1.23 (XTAL2), Y1.4
- new net: C_CLK1.1, U1.24 (XTAL1), Y1.1
- new net: R_USB3.1, U1.4 (D-)
- new net: R_HWB.2, U1.43 ((ALE/~HWB~)PE2)
- new net: R_USB4.1, U1.5 (D+)
- new net: C_REF.1, U1.62 (AREF)
- new net: C_CAP.1, U1.7 (UCAP)
- new net: J1.A5 (CC1), R_USB1.1
- new net: J1.A6 (D+), J1.B6 (D+), R_USB4.2
- new net: J1.A7 (D-), J1.B7 (D-), R_USB3.2
- new net: J1.B5 (CC2), R_USB2.1
- new net GND: C_AVCC.2, C_CAP.2, C_CLK1.2, C_CLK2.2, C_REF.2, C_UVCC.2, C_VCC1.2, C_VCC2.2, J1.A1 (GND), J1.A12 (GND), J1.B1 (GND), J1.B12 (GND), J1.S1 (SHIELD), R_HWB.1, R_USB1.2, R_USB2.2, SW1.1, U1.22 (GND), U1.53 (GND), U1.6 (UGND), U1.63 (GND), Y1.2, Y1.3
- new net VCC: C_AVCC.1, C_UVCC.1, C_VCC1.1, C_VCC2.1, J1.A4 (VBUS), J1.A9 (VBUS), J1.B4 (VBUS), J1.B9 (VBUS), R_RST.2, U1.21 (VCC), U1.3 (UVCC), U1.52 (VCC), U1.64 (AVCC), U1.8 (VBUS)
- new net col00: U1.28 ((TXD1/INT3)PD3)
- new net col01: U1.29 ((ICP1)PD4)
- new net col02: U1.30 ((XCK1)PD5)
- new net col03: U1.31 ((T1)PD6)
- new net col04: U1.32 ((T0)PD7)
- new net col05: U1.35 ((A8)PC0)
- new net col06: U1.36 ((A9)PC1)
- new net col07: U1.37 ((A10)PC2)
- new net col08: U1.38 ((A11/T.3)PC3)
- new net col09: U1.39 ((A12/OC.3C)PC4)
- new net col10: U1.40 ((A13/OC.3B)PC5)
- new net col11: U1.41 ((A14/OC.3A)PC6)
- new net col12: U1.42 ((A15/IC.3/CLKO)PC7)
- new net col13: U1.54 ((ADC7/TDI)PF7)
- new net col14: U1.55 ((ADC6/TDO)PF6)
- new net col15: U1.56 ((ADC6/TMS)PF5)
- new net col16: U1.57 ((ADC5/TCK)PF4)
- new net col17: U1.58 ((ADC3)PF3)
- new net col18: U1.59 ((ADC2)PF2)
- new net col19: U1.60 ((ADC1)PF1)
- new net col20: U1.61 ((ADC0)PF0)
- new net row0: U1.48 ((AD3)PA3)
- new net row1: U1.47 ((AD4)PA4)
- new net row2: U1.46 ((AD5)PA5)
- new net row3: U1.45 ((AD6)PA6)
- new net row4: U1.44 ((AD7)PA7)
- no-connect marks 0 -> 31

Commit message: 2017.11.14 Update
- Redid schematic and layout
- Now using USB-C connector
Parts:
- removed Y1: 16M, symbol Crystal_GND23
- added D0,1, D0,10, D0,11, D0,12, D0,13, D0,14, D0,15, D0,16, D0,17, D0,18, D0,19, D0,2, D0,20, D0,21, D0,3, D0,4, D0,5, D0,6, D0,7, D0,8, D0,9, D1,1, D1,10, D1,11, D1,12, D1,13, D1,14, D1,15, D1,16, D1,17, D1,18, D1,19, D1,2, D1,20, D1,21, D1,3, D1,4, D1,5, D1,6, D1,7, D1,8, D1,9, D2,1, D2,10, D2,11, D2,12, D2,13, D2,14, D2,15, D2,16, D2,17, D2,18, D2,19, D2,2, D2,3, D2,4, D2,5, D2,6, D2,7, D2,8, D2,9, D3,1, D3,10, D3,11, D3,12, D3,13, D3,14, D3,15, D3,16, D3,17, D3,18, D3,19, D3,2, D3,3, D3,4, D3,5, D3,6, D3,7, D3,8, D3,9, D4,1, D4,10, D4,11, D4,12, D4,13, D4,2, D4,3, D4,4, D4,5, D4,6, D4,7, D4,8, D4,9: D, keyboard_parts:D_SOD123_axial, symbol D
- added K0,1, K0,10, K0,11, K0,12, K0,13, K0,14, K0,15, K0,16, K0,17, K0,19, K0,2, K0,20, K0,21, K0,3, K0,4, K0,5, K0,6, K0,7, K0,8, K0,9, K1,1, K1,10, K1,11, K1,12, K1,13, K1,14, K1,15, K1,16, K1,17, K1,19, K1,2, K1,20, K1,21, K1,3, K1,6, K1,7, K1,8, K1,9, K2,1, K2,10, K2,11, K2,12, K2,13, K2,14, K2,15, K2,17, K2,18, K2,19, K2,2, K2,3, K2,5, K2,6, K2,7, K2,8, K2,9, K3,1, K3,10, K3,11, K3,12, K3,13, K3,14, K3,15, K3,17, K3,18, K3,19, K3,2, K3,3, K3,6, K3,7, K3,8, K3,9, K4,11, K4,12, K4,13, K4,2: KEYSW, keebs:Mx_Alps_100, symbol KEYSW
- added K0,18, K1,4, K3,4, K4,1: KEYSW, keebs:Mx_Alps_200, symbol KEYSW
- added K1,18, K1,5: KEYSW, keebs:Mx_Alps_150, symbol KEYSW
- added K2,16, K3,5: KEYSW, keebs:Mx_Alps_225, symbol KEYSW
- added K2,4: KEYSW, keebs:Mx_Alps_175, symbol KEYSW
- added K3,16: KEYSW, keebs:Mx_Alps_275, symbol KEYSW
- added K4,10, K4,3, K4,4, K4,5, K4,7, K4,8, K4,9: KEYSW, keebs:Mx_Alps_125, symbol KEYSW
- added K4,6: KEYSW, keebs:Mx_Alps_625, symbol KEYSW
- added Y1: 16M, Crystals:Crystal_SMD_SeikoEpson_FA238-4pin_3.2x2.5mm_HandSoldering, symbol Crystal_GND24
- C_AVCC1: renamed from C_AVCC; footprint (none) -> Capacitors_SMD:C_0805_HandSoldering
- C_CAP1: renamed from C_CAP; footprint (none) -> Capacitors_SMD:C_0805_HandSoldering
- C_CLK1, C_CLK2, C_VCC1, C_VCC2: footprint (none) -> Capacitors_SMD:C_0805_HandSoldering
- C_REF1: renamed from C_REF; footprint (none) -> Capacitors_SMD:C_0805_HandSoldering
- C_UVCC1: renamed from C_UVCC; footprint (none) -> Capacitors_SMD:C_0805_HandSoldering
- J1: footprint (none) -> Connectors_USB:USB_C_Receptacle_Amphenol_12401610E4-2A
- R_HWB1: renamed from R_HWB; footprint (none) -> Resistors_SMD:R_0805_HandSoldering
- R_RST1: renamed from R_RST; footprint (none) -> Resistors_SMD:R_0805_HandSoldering
- R_USB1, R_USB2, R_USB3, R_USB4: footprint (none) -> Resistors_SMD:R_0805_HandSoldering
- SW1: footprint (none) -> Buttons_Switches_SMD:SW_SPST_TL3342
- U1: footprint (none) -> Housings_QFP:TQFP-64_14x14mm_Pitch0.8mm
Connections:
- net GND: now also Y1.2, Y1.4
- net col00: now also K0,1.1, K1,1.1, K2,1.1, K3,1.1, K4,1.1
- net col01: now also K0,2.1, K1,2.1, K2,2.1, K3,2.1
- net col02: now also K0,3.1, K1,3.1, K2,3.1, K3,3.1, K4,2.1
- net col03: now also K0,4.1, K1,4.1, K3,4.1
- net col04: now also K0,5.1, K1,5.1, K2,4.1, K3,5.1, K4,3.1
- net col05: now also K0,6.1, K1,6.1, K2,5.1, K3,6.1, K4,4.1
- net col06: now also K0,7.1, K1,7.1, K2,6.1, K3,7.1, K4,5.1
- net col07: now also K0,8.1, K1,8.1, K2,7.1, K3,8.1
- net col08: now also K0,9.1, K1,9.1, K2,8.1, K3,9.1
- net col09: now also K0,10.1, K1,10.1, K2,9.1, K3,10.1, K4,6.1
- net col10: now also K0,11.1, K1,11.1, K2,10.1, K3,11.1
- net col11: now also K0,12.1, K1,12.1, K2,11.1, K3,12.1
- net col12: now also K0,13.1, K1,13.1, K2,12.1, K3,13.1
- net col13: now also K0,14.1, K1,14.1, K2,13.1, K3,14.1, K4,7.1
- net col14: now also K0,15.1, K1,15.1, K2,14.1, K3,15.1, K4,8.1
- net col15: now also K0,16.1, K1,16.1, K2,15.1
- net col16: now also K0,17.1, K1,17.1, K3,16.1, K4,9.1
- net col17: now also K0,18.1, K1,18.1, K2,16.1, K4,10.1
- net col18: now also K0,19.1, K1,19.1, K2,17.1, K3,17.1, K4,11.1
- net col19: now also K0,20.1, K1,20.1, K2,18.1, K3,18.1, K4,12.1
- net col20: now also K0,21.1, K1,21.1, K2,19.1, K3,19.1, K4,13.1
- net row0: now also D0,1.1, D0,10.1, D0,11.1, D0,12.1, D0,13.1, D0,14.1, D0,15.1, D0,16.1, D0,17.1, D0,18.1, D0,19.1, D0,2.1, D0,20.1, D0,21.1, D0,3.1, D0,4.1, D0,5.1, D0,6.1, D0,7.1, D0,8.1, D0,9.1
- net row1: now also D1,1.1, D1,10.1, D1,11.1, D1,12.1, D1,13.1, D1,14.1, D1,15.1, D1,16.1, D1,17.1, D1,18.1, D1,19.1, D1,2.1, D1,20.1, D1,21.1, D1,3.1, D1,4.1, D1,5.1, D1,6.1, D1,7.1, D1,8.1, D1,9.1
- net row2: now also D2,1.1, D2,10.1, D2,11.1, D2,12.1, D2,13.1, D2,14.1, D2,15.1, D2,16.1, D2,17.1, D2,18.1, D2,19.1, D2,2.1, D2,3.1, D2,4.1, D2,5.1, D2,6.1, D2,7.1, D2,8.1, D2,9.1
- net row3: now also D3,1.1, D3,10.1, D3,11.1, D3,12.1, D3,13.1, D3,14.1, D3,15.1, D3,16.1, D3,17.1, D3,18.1, D3,19.1, D3,2.1, D3,3.1, D3,4.1, D3,5.1, D3,6.1, D3,7.1, D3,8.1, D3,9.1
- net row4: now also D4,1.1, D4,10.1, D4,11.1, D4,12.1, D4,13.1, D4,2.1, D4,3.1, D4,4.1, D4,5.1, D4,6.1, D4,7.1, D4,8.1, D4,9.1
- net at C_CLK2.1, U1.23 (XTAL2): now also Y1.3
- net at C_CLK1.1, U1.24 (XTAL1): now also Y1.1
- new net: D0,1.2, K0,1.2
- new net: D0,2.2, K0,2.2
- new net: D0,3.2, K0,3.2
- new net: D0,4.2, K0,4.2
- new net: D0,5.2, K0,5.2
- new net: D0,6.2, K0,6.2
- new net: D0,7.2, K0,7.2
- new net: D0,8.2, K0,8.2
- new net: D0,9.2, K0,9.2
- new net: D0,10.2, K0,10.2
- new net: D0,11.2, K0,11.2
- new net: D0,12.2, K0,12.2
- new net: D0,13.2, K0,13.2
- new net: D0,14.2, K0,14.2
- new net: D0,15.2, K0,15.2
- new net: D0,16.2, K0,16.2
- new net: D0,17.2, K0,17.2
- new net: D0,18.2, K0,18.2
- new net: D0,19.2, K0,19.2
- new net: D0,20.2, K0,20.2
- new net: D0,21.2, K0,21.2
- new net: D1,1.2, K1,1.2
- new net: D1,2.2, K1,2.2
- new net: D1,3.2, K1,3.2
- new net: D1,4.2, K1,4.2
- new net: D1,5.2, K1,5.2
- new net: D1,6.2, K1,6.2
- new net: D1,7.2, K1,7.2
- new net: D1,8.2, K1,8.2
- new net: D1,9.2, K1,9.2
- new net: D1,10.2, K1,10.2
- new net: D1,11.2, K1,11.2
- new net: D1,12.2, K1,12.2
- new net: D1,13.2, K1,13.2
- new net: D1,14.2, K1,14.2
- new net: D1,15.2, K1,15.2
- new net: D1,16.2, K1,16.2
- new net: D1,17.2, K1,17.2
- new net: D1,18.2, K1,18.2
- new net: D1,19.2, K1,19.2
- new net: D1,20.2, K1,20.2
- new net: D1,21.2, K1,21.2
- new net: D2,1.2, K2,1.2
- new net: D2,2.2, K2,2.2
- new net: D2,3.2, K2,3.2
- new net: D2,4.2, K2,4.2
- new net: D2,5.2, K2,5.2
- new net: D2,6.2, K2,6.2
- new net: D2,7.2, K2,7.2
- new net: D2,8.2, K2,8.2
- new net: D2,9.2, K2,9.2
- new net: D2,10.2, K2,10.2
- new net: D2,11.2, K2,11.2
- new net: D2,12.2, K2,12.2
- new net: D2,13.2, K2,13.2
- new net: D2,14.2, K2,14.2
- new net: D2,15.2, K2,15.2
- new net: D2,16.2, K2,16.2
- new net: D2,17.2, K2,17.2
- new net: D2,18.2, K2,18.2
- new net: D2,19.2, K2,19.2
- new net: D3,1.2, K3,1.2
- new net: D3,2.2, K3,2.2
- new net: D3,3.2, K3,3.2
- new net: D3,4.2, K3,4.2
- new net: D3,5.2, K3,5.2
- new net: D3,6.2, K3,6.2
- new net: D3,7.2, K3,7.2
- new net: D3,8.2, K3,8.2
- new net: D3,9.2, K3,9.2
- new net: D3,10.2, K3,10.2
- new net: D3,11.2, K3,11.2
- new net: D3,12.2, K3,12.2
- new net: D3,13.2, K3,13.2
- new net: D3,14.2, K3,14.2
- new net: D3,15.2, K3,15.2
- new net: D3,16.2, K3,16.2
- new net: D3,17.2, K3,17.2
- new net: D3,18.2, K3,18.2
- new net: D3,19.2, K3,19.2
- new net: D4,1.2, K4,1.2
- new net: D4,2.2, K4,2.2
- new net: D4,3.2, K4,3.2
- new net: D4,4.2, K4,4.2
- new net: D4,5.2, K4,5.2
- new net: D4,6.2, K4,6.2
- new net: D4,7.2, K4,7.2
- new net: D4,8.2, K4,8.2
- new net: D4,9.2, K4,9.2
- new net: D4,10.2, K4,10.2
- new net: D4,11.2, K4,11.2
- new net: D4,12.2, K4,12.2
- new net: D4,13.2, K4,13.2
Other:
- moved on the sheet: C_AVCC1, C_CAP1, C_CLK1, C_CLK2, C_REF1, C_UVCC1, C_VCC1, C_VCC2, J1, R_HWB1, R_RST1, R_USB1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

Commit message: 2017.11.15 Update
- Layed out most electronics on the board
Parts:
- Y1: footprint Crystals:Crystal_SMD_SeikoEpson_FA238-4pin_3.2x2.5mm_HandSoldering -> Crystals:Crystal_SMD_SeikoEpson_FA238-4pin_3.2x2.5mm
Changed lines of the file:
@@
 F 0 "Y1" V 3150 3200 50  0000 L CNN
 F 1 "16M" V 3150 3400 50  0000 L CNN
-F 2 "Crystals:Crystal_SMD_SeikoEpson_FA238-4pin_3.2x2.5mm_HandSoldering" H 3350 3350 50  0001 C CNN
+F 2 "Crystals:Crystal_SMD_SeikoEpson_FA238-4pin_3.2x2.5mm" H 3350 3350 50  0001 C CNN
 F 3 "" H 3350 3350 50  0001 C CNN
 	1    3350 3350

Commit message: 2018.03.15 Update
- Updated labels on switches and diodes to better match array subscripts
- Started preliminary C code for the firmware
Parts:
- renumbered D0,1 to D0,0, D0,2 to D0,1, D0,11 to D0,10, D0,12 to D0,11, D0,13 to D0,12, D0,14 to D0,13, D0,15 to D0,14, D0,16 to D0,15, D0,17 to D0,16, D0,18 to D0,17, D0,19 to D0,18, D0,20 to D0,19, D0,3 to D0,2, D0,21 to D0,20, D0,4 to D0,3, D0,5 to D0,4, D0,6 to D0,5, D0,7 to D0,6, D0,8 to D0,7, D0,9 to D0,8, D0,10 to D0,9, D1,1 to D1,0, D1,2 to D1,1, D1,11 to D1,10, D1,12 to D1,11, D1,13 to D1,12, D1,14 to D1,13, D1,15 to D1,14, D1,16 to D1,15, D1,17 to D1,16, D1,18 to D1,17, D1,19 to D1,18, D1,20 to D1,19, D1,3 to D1,2, D1,21 to D1,20, D1,4 to D1,3, D1,5 to D1,4, D1,6 to D1,5, D1,7 to D1,6, D1,8 to D1,7, D1,9 to D1,8, D1,10 to D1,9, D2,1 to D2,0, D2,2 to D2,1, D2,16 to D2,17, D2,17 to D2,18, D2,18 to D2,19, D2,3 to D2,2, D2,19 to D2,20, D3,1 to D3,0, D3,2 to D3,1, D3,11 to D3,10, D3,12 to D3,11, D3,13 to D3,12, D3,14 to D3,13, D3,15 to D3,14, D3,17 to D3,18, D3,18 to D3,19, D3,3 to D3,2, D3,19 to D3,20, D3,4 to D3,3, D3,5 to D3,4, D3,6 to D3,5, D3,7 to D3,6, D3,8 to D3,7, D3,9 to D3,8, D3,10 to D3,9, D4,1 to D4,0, D4,7 to D4,13, D4,8 to D4,14, D4,9 to D4,16, D4,10 to D4,17, D4,11 to D4,18, D4,12 to D4,19, D4,13 to D4,20, D4,3 to D4,4, D4,4 to D4,5, D4,5 to D4,6, D4,6 to D4,9, K0,1 to K0,0, K0,2 to K0,1, K0,11 to K0,10, K0,12 to K0,11, K0,13 to K0,12, K0,14 to K0,13, K0,15 to K0,14, K0,16 to K0,15, K0,17 to K0,16, K0,18 to K0,17, K0,19 to K0,18, K0,20 to K0,19, K0,3 to K0,2, K0,21 to K0,20, K0,4 to K0,3, K0,5 to K0,4, K0,6 to K0,5, K0,7 to K0,6, K0,8 to K0,7, K0,9 to K0,8, K0,10 to K0,9, K1,1 to K1,0, K1,2 to K1,1, K1,11 to K1,10, K1,12 to K1,11, K1,13 to K1,12, K1,14 to K1,13, K1,15 to K1,14, K1,16 to K1,15, K1,17 to K1,16, K1,18 to K1,17, K1,19 to K1,18, K1,20 to K1,19, K1,3 to K1,2, K1,21 to K1,20, K1,4 to K1,3, K1,5 to K1,4, K1,6 to K1,5, K1,7 to K1,6, K1,8 to K1,7, K1,9 to K1,8, K1,10 to K1,9, K2,1 to K2,0, K2,2 to K2,1, K2,16 to K2,17, K2,17 to K2,18, K2,18 to K2,19, K2,3 to K2,2, K2,19 to K2,20, K3,1 to K3,0, K3,2 to K3,1, K3,11 to K3,10, K3,12 to K3,11, K3,13 to K3,12, K3,14 to K3,13, K3,15 to K3,14, K3,17 to K3,18, K3,18 to K3,19, K3,3 to K3,2, K3,19 to K3,20, K3,4 to K3,3, K3,5 to K3,4, K3,6 to K3,5, K3,7 to K3,6, K3,8 to K3,7, K3,9 to K3,8, K3,10 to K3,9, K4,1 to K4,0, K4,7 to K4,13, K4,8 to K4,14, K4,9 to K4,16, K4,10 to K4,17, K4,11 to K4,18, K4,12 to K4,19, K4,13 to K4,20, K4,3 to K4,4, K4,4 to K4,5, K4,5 to K4,6, K4,6 to K4,9
Other:
- moved on the sheet: D0,0, D0,1, D0,10, D0,11, D0,12, D0,13, D0,14, D0,15, D0,16, D0,17, D0,18, D0,19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

Commit message: 2018.04.16 Nightly
Other:
- moved on the sheet: C_AVCC1, C_CLK1, C_CLK2, C_UVCC1, C_VCC1, C_VCC2, Y1

Commit message: 2018.04.27 Update
- Version 1.1 Release
- Cleaned up routing to the USB port
- Made seperate schematic sheet with key matrix (so it can be used in JayKey2)
Parts:
- removed D0,0, D0,1, D0,10, D0,11, D0,12, D0,13, D0,14, D0,15, D0,16, D0,17, D0,18, D0,19, D0,2, D0,20, D0,3, D0,4, D0,5, D0,6, D0,7, D0,8, D0,9, D1,0, D1,1, D1,10, D1,11, D1,12, D1,13, D1,14, D1,15, D1,16, D1,17, D1,18, D1,19, D1,2, D1,20, D1,3, D1,4, D1,5, D1,6, D1,7, D1,8, D1,9, D2,0, D2,1, D2,10, D2,11, D2,12, D2,13, D2,14, D2,15, D2,17, D2,18, D2,19, D2,2, D2,20, D2,4, D2,5, D2,6, D2,7, D2,8, D2,9, D3,0, D3,1, D3,10, D3,11, D3,12, D3,13, D3,14, D3,16, D3,18, D3,19, D3,2, D3,20, D3,3, D3,4, D3,5, D3,6, D3,7, D3,8, D3,9, D4,0, D4,13, D4,14, D4,16, D4,17, D4,18, D4,19, D4,2, D4,20, D4,4, D4,5, D4,6, D4,9: D, keyboard_parts:D_SOD123_axial, symbol D
- removed K0,0, K0,1, K0,10, K0,11, K0,12, K0,13, K0,14, K0,15, K0,16, K0,18, K0,19, K0,2, K0,20, K0,3, K0,4, K0,5, K0,6, K0,7, K0,8, K0,9, K1,0, K1,1, K1,10, K1,11, K1,12, K1,13, K1,14, K1,15, K1,16, K1,18, K1,19, K1,2, K1,20, K1,5, K1,6, K1,7, K1,8, K1,9, K2,0, K2,1, K2,10, K2,11, K2,12, K2,13, K2,14, K2,15, K2,18, K2,19, K2,2, K2,20, K2,5, K2,6, K2,7, K2,8, K2,9, K3,0, K3,1, K3,10, K3,11, K3,12, K3,13, K3,14, K3,18, K3,19, K3,2, K3,20, K3,5, K3,6, K3,7, K3,8, K3,9, K4,18, K4,19, K4,2, K4,20: KEYSW, keebs:Mx_Alps_100, symbol KEYSW
- removed K0,17, K1,3, K3,3, K4,0: KEYSW, keebs:Mx_Alps_200, symbol KEYSW
- removed K1,17, K1,4: KEYSW, keebs:Mx_Alps_150, symbol KEYSW
- removed K2,17, K3,4: KEYSW, keebs:Mx_Alps_225, symbol KEYSW
- removed K2,4: KEYSW, keebs:Mx_Alps_175, symbol KEYSW
- removed K3,16: KEYSW, keebs:Mx_Alps_275, symbol KEYSW
- removed K4,13, K4,14, K4,16, K4,17, K4,4, K4,5, K4,6: KEYSW, keebs:Mx_Alps_125, symbol KEYSW
- removed K4,9: KEYSW, keebs:Mx_Alps_625, symbol KEYSW
Other:
- moved on the sheet: C_AVCC1, C_CAP1, C_CLK1, C_CLK2, C_REF1, C_UVCC1, C_VCC1, C_VCC2, J1, R_HWB1, R_RST1, R_USB1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

Commit message: 2018.08.27 Nightly
Parts:
- added C_VBUS1: 10u, Capacitors_SMD:C_0805_HandSoldering, symbol C
- added J2: USB_C_Receptacle, Connectors_USB:USB_C_Receptacle_Amphenol_12401610E4-2A, symbol USB_C_Receptacle
- added R_USB5, R_USB6: 5.1k, Resistors_SMD:R_0805_HandSoldering, symbol R
- added R_USB7, R_USB8: 22, Resistors_SMD:R_0805_HandSoldering, symbol R
Connections:
- net GND: now also C_VBUS1.2, J2.A1 (GND), J2.A12 (GND), J2.B1 (GND), J2.B12 (GND), J2.S1 (SHIELD), R_USB5.2, R_USB6.2
- net VCC: now also C_VBUS1.1, J2.A4 (VBUS), J2.A9 (VBUS), J2.B4 (VBUS), J2.B9 (VBUS)
- net at J1.A6 (D+), J1.B6 (D+), R_USB4.2: now also R_USB8.1
- net at J1.A7 (D-), J1.B7 (D-), R_USB3.2: now also R_USB7.1
- new net: J2.A5 (CC1), R_USB5.1
- new net: J2.A6 (D+), J2.B6 (D+), R_USB8.2
- new net: J2.A7 (D-), J2.B7 (D-), R_USB7.2
- new net: J2.B5 (CC2), R_USB6.1
- no-connect marks 31 -> 41
