File: PCB/JayKey1.sch (KiCad schematic (older format))
At the start: 24 parts, among them J1 USB_C_Receptacle, J2 USB_C_Receptacle, SW1 SW_PUSH, U1 AT90USB1286, Y1 16M

Commit message: 2018.08.28 Nightly
Parts:
- added C_VBUS2: 10u, Capacitors_SMD:C_0805_HandSoldering, symbol C
- added D_VBUS1, D_VBUS2: D, keyboard_parts:D_SOD123_axial, symbol D
- R_RST1: value 10k -> 47k
Connections:
- net GND: now also C_VBUS2.2
- net DMINUS: now reaches R_USB3.1, U1.4 (D-)
- net DMINUS: now also R_USB7.1
- net DPLUS: now reaches R_USB4.1, U1.5 (D+)
- net DPLUS: now also R_USB8.1
- net at J1.A6 (D+), J1.B6 (D+), R_USB4.2: no longer R_USB8.1
- net at J1.A7 (D-), J1.B7 (D-), R_USB3.2: no longer R_USB7.1
- net VCC renamed VBUS
- net VBUS: now also C_VBUS2.1, D_VBUS1.1, D_VBUS2.1; no longer J1.A4 (VBUS), J1.A9 (VBUS), J1.B4 (VBUS), J1.B9 (VBUS), J2.A4 (VBUS), J2.A9 (VBUS), J2.B4 (VBUS), J2.B9 (VBUS)
- new net: D_VBUS1.2, J1.A4 (VBUS), J1.A9 (VBUS), J1.B4 (VBUS), J1.B9 (VBUS)
- new net: D_VBUS2.2, J2.A4 (VBUS), J2.A9 (VBUS), J2.B4 (VBUS), J2.B9 (VBUS)
Other:
- note added: "Left USB Port"
- note added: "Right USB Port"
- moved on the sheet: C_AVCC1, C_CAP1, C_CLK1, C_CLK2, C_REF1, C_UVCC1, C_VCC1, C_VCC2, J1, J2, R_HWB1, R_RST1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

Commit message: 2018.09.23 Nightly
Parts:
- removed C_VBUS1, C_VBUS2: 10u, Capacitors_SMD:C_0805_HandSoldering, symbol C
- removed D_VBUS1, D_VBUS2: D, keyboard_parts:D_SOD123_axial, symbol D
- removed J1, J2: USB_C_Receptacle, Connectors_USB:USB_C_Receptacle_Amphenol_12401610E4-2A, symbol USB_C_Receptacle
- removed R_USB1, R_USB2, R_USB5, R_USB6: 5.1k, Resistors_SMD:R_0805_HandSoldering, symbol R
- removed R_USB3, R_USB4, R_USB7, R_USB8: 22, Resistors_SMD:R_0805_HandSoldering, symbol R
- removed U1: AT90USB1286, Housings_QFP:TQFP-64_14x14mm_Pitch0.8mm, symbol AT90USB1286
- added U1: AT90USB1286-AU, Housings_QFP:TQFP-64_14x14mm_Pitch0.8mm, symbol AT90USB1286-AU
- renumbered C_REF1 to C_AREF1, C_CAP1 to C_UCAP1
Connections:
- wire segments 73 -> 41
- no-connect marks 41 -> 21
Other:
- note removed: "Left USB Port"
- note removed: "Right USB Port"
- moved on the sheet: C_AREF1, C_AVCC1, C_CLK1, C_CLK2, C_UCAP1, C_UVCC1, C_VCC1, C_VCC2, R_HWB1, R_RST1, SW1, Y1

Commit message: 2018.09.25 Nightly
Parts:
- added C_VBUS1: 10u, symbol C
- added R_USB1, R_USB2: 22, symbol R
- C_UVCC1: value 1u -> 100n
Connections:
- net labels added: VCC
- net labels removed: VBUS
- wire segments 41 -> 46
Other:
- moved on the sheet: C_AREF1, C_AVCC1, C_UCAP1, C_UVCC1, C_VCC1, C_VCC2, R_HWB1

Commit message: 2018.09.29 Nightly
Parts:
- C_VBUS1: footprint (none) -> Capacitors_SMD:C_0805_HandSoldering
- R_USB1, R_USB2: footprint (none) -> Resistors_SMD:R_0805_HandSoldering
Changed lines of the file:
@@
 $EndComp
 $Comp
-L GND #PWR03
+L GND #PWR01
 U 1 1 5A0B3FFB
 P 3600 2200
-F 0 "#PWR03" H 3600 1950 50  0001 C CNN
+F 0 "#PWR01" H 3600 1950 50  0001 C CNN
 F 1 "GND" H 3600 2050 50  0000 C CNN
 F 2 "" H 3600 2200 50  0001 C CNN
@@
 $EndComp
 $Comp
-L GND #PWR04
+L GND #PWR02
 U 1 1 5A0B403C
 P 3350 2900
-F 0 "#PWR04" H 3350 2650 50  0001 C CNN
+F 0 "#PWR02" H 3350 2650 50  0001 C CNN
 F 1 "GND" H 3350 2750 50  0000 C CNN
 F 2 "" H 3350 2900 50  0001 C CNN
@@
 $EndComp
 $Comp
-L GND #PWR05
+L GND #PWR03
 U 1 1 5A0B406B
 P 3850 2900
-F 0 "#PWR05" H 3850 2650 50  0001 C CNN
+F 0 "#PWR03" H 3850 2650 50  0001 C CNN
 F 1 "GND" H 3850 2750 50  0000 C CNN
 F 2 "" H 3850 2900 50  0001 C CNN
@@
 $EndComp
 $Comp
-L GND #PWR06
+L GND #PWR04
 U 1 1 5A0B42A8
 P 3600 2600
-F 0 "#PWR06" H 3600 2350 50  0001 C CNN
+F 0 "#PWR04" H 3600 2350 50  0001 C CNN
 F 1 "GND" H 3600 2450 50  0000 C CNN
 F 2 "" H 3600 2600 50  0001 C CNN
@@
 $EndComp
 $Comp
-L GND #PWR07
+L GND #PWR05
 U 1 1 5A0B4CA7
 P 4500 3600
-F 0 "#PWR07" H 4500 3350 50  0001 C CNN
+F 0 "#PWR05" H 4500 3350 50  0001 C CNN
 F 1 "GND" H 4500 3450 50  0000 C CNN
 F 2 "" H 4500 3600 50  0001 C CNN
@@
 $EndComp
 $Comp
-L GND #PWR08
+L GND #PWR06
 U 1 1 5A0B4F28
 P 6400 5350
-F 0 "#PWR08" H 6400 5100 50  0001 C CNN
+F 0 "#PWR06" H 6400 5100 50  0001 C CNN
 F 1 "GND" H 6400 5200 50  0000 C CNN
 F 2 "" H 6400 5350 50  0001 C CNN
@@
 $EndComp
 $Comp
-L GND #PWR09
+L GND #PWR07
 U 1 1 5A0B4F5A
 P 6500 5350
-F 0 "#PWR09" H 6500 5100 50  0001 C CNN
+F 0 "#PWR07" H 6500 5100 50  0001 C CNN
 F 1 "GND" H 6500 5200 50  0000 C CNN
 F 2 "" H 6500 5350 50  0001 C CNN
@@
 $EndComp
 $Comp
-L GND #PWR010
+L GND #PWR08
 U 1 1 5A0B4F8C
 P 6600 5350
-F 0 "#PWR010" H 6600 5100 50  0001 C CNN
+F 0 "#PWR08" H 6600 5100 50  0001 C CNN
 F 1 "GND" H 6600 5200 50  0000 C CNN
 F 2 "" H 6600 5350 50  0001 C CNN
@@
 $EndComp
 $Comp
-L GND #PWR015
+L GND #PWR09
 U 1 1 5A0B5542
 P 5150 2650
-F 0 "#PWR015" H 5150 2400 50  0001 C CNN
+F 0 "#PWR09" H 5150 2400 50  0001 C CNN
 F 1 "GND" H 5150 2500 50  0000 C CNN
 F 2 "" H 5150 2650 50  0001 C CNN
@@
 $EndComp
 $Comp
-L GND #PWR016
+L GND #PWR010
 U 1 1 5A0B55F6
 P 4200 3600
-F 0 "#PWR016" H 4200 3350 50  0001 C CNN
+F 0 "#PWR010" H 4200 3350 50  0001 C CNN
 F 1 "GND" H 4200 3450 50  0000 C CNN
 F 2 "" H 4200 3600 50  0001 C CNN
@@
 $EndComp
 $Comp
-L GND #PWR017
+L GND #PWR011
 U 1 1 5A0B60A2
 P 4800 5100
-F 0 "#PWR017" H 4800 4850 50  0001 C CNN
+F 0 "#PWR011" H 4800 4850 50  0001 C CNN
 F 1 "GND" H 4800 4950 50  0000 C CNN
 F 2 "" H 4800 5100 50  0001 C CNN
@@
 $EndComp
 $Comp
-L GND #PWR018
+L GND #PWR012
 U 1 1 5A0B6DE3
 P 6050 6200
-F 0 "#PWR018" H 6050 5950 50  0001 C CNN
+F 0 "#PWR012" H 6050 5950 50  0001 C CNN
 F 1 "GND" H 6050 6050 50  0000 C CNN
 F 2 "" H 6050 6200 50  0001 C CNN
@@
 $EndComp
 $Comp
-L GND #PWR019
+L GND #PWR013
 U 1 1 5A0B71F2
 P 6500 6200
-F 0 "#PWR019" H 6500 5950 50  0001 C CNN
+F 0 "#PWR013" H 6500 5950 50  0001 C CNN
 F 1 "GND" H 6500 6050 50  0000 C CNN
 F 2 "" H 6500 6200 50  0001 C CNN
@@
 $EndComp
 $Comp
-L GND #PWR020
+L GND #PWR014
 U 1 1 5A0B7236
 P 6950 6200
-F 0 "#PWR020" H 6950 5950 50  0001 C CNN
+F 0 "#PWR014" H 6950 5950 50  0001 C CNN
 F 1 "GND" H 6950 6050 50  0000 C CNN
 F 2 "" H 6950 6200 50  0001 C CNN
@@
 $EndComp
 $Comp
-L GND #PWR021
+L GND #PWR015
 U 1 1 5A0B727A
 P 7400 6200
-F 0 "#PWR021" H 7400 5950 50  0001 C CNN
+F 0 "#PWR015" H 7400 5950 50  0001 C CNN
 F 1 "GND" H 7400 6050 50  0000 C CNN
 F 2 "" H 7400 6200 50  0001 C CNN
@@
 $EndComp
 $Comp
-L GND #PWR022
+L GND #PWR016
 U 1 1 5A0B8008
 P 4350 1750
-F 0 "#PWR022" H 4350 1500 50  0001 C CNN
+F 0 "#PWR016" H 4350 1500 50  0001 C CNN
 F 1 "GND" H 4350 1600 50  0000 C CNN
 F 2 "" H 4350 1750 50  0001 C CNN
@@
 DPLUS
 $Comp
-L VCC #PWR?
+L VCC #PWR017
 U 1 1 5BAAD93C
 P 6400 1400
-F 0 "#PWR?" H 6400 1250 50  0001 C CNN
+F 0 "#PWR017" H 6400 1250 50  0001 C CNN
 F 1 "VCC" H 6400 1550 50  0000 C CNN
 F 2 "" H 6400 1400 50  0001 C CNN
@@
 $EndComp
 $Comp
-L VCC #PWR?
+L VCC #PWR018
 U 1 1 5BAAD9A4
 P 6500 1400
-F 0 "#PWR?" H 6500 1250 50  0001 C CNN
+F 0 "#PWR018" H 6500 1250 50  0001 C CNN
 F 1 "VCC" H 6500 1550 50  0000 C CNN
 F 2 "" H 6500 1400 50  0001 C CNN
@@
 $EndComp
 $Comp
-L VCC #PWR?
+L VCC #PWR019
 U 1 1 5BAADA0C
 P 6600 1400
-F 0 "#PWR?" H 6600 1250 50  0001 C CNN
+F 0 "#PWR019" H 6600 1250 50  0001 C CNN
 F 1 "VCC" H 6600 1550 50  0000 C CNN
 F 2 "" H 6600 1400 50  0001 C CNN
@@
 $EndComp
 $Comp
-L VCC #PWR?
+L VCC #PWR020
 U 1 1 5BAADA98
 P 6050 5800
-F 0 "#PWR?" H 6050 5650 50  0001 C CNN
+F 0 "#PWR020" H 6050 5650 50  0001 C CNN
 F 1 "VCC" H 6050 5950 50  0000 C CNN
 F 2 "" H 6050 5800 50  0001 C CNN
@@
 $EndComp
 $Comp
-L VCC #PWR?
+L VCC #PWR021
 U 1 1 5BAADB00
 P 6500 5800
-F 0 "#PWR?" H 6500 5650 50  0001 C CNN
+F 0 "#PWR021" H 6500 5650 50  0001 C CNN
 F 1 "VCC" H 6500 5950 50  0000 C CNN
 F 2 "" H 6500 5800 50  0001 C CNN
@@
 $EndComp
 $Comp
-L VCC #PWR?
+L VCC #PWR022
 U 1 1 5BAADB68
 P 6950 5800
-F 0 "#PWR?" H 6950 5650 50  0001 C CNN
+F 0 "#PWR022" H 6950 5650 50  0001 C CNN
 F 1 "VCC" H 6950 5950 50  0000 C CNN
 F 2 "" H 6950 5800 50  0001 C CNN
@@
 $EndComp
 $Comp
-L VCC #PWR?
+L VCC #PWR023
 U 1 1 5BAADBD0
 P 7400 5800
-F 0 "#PWR?" H 7400 5650 50  0001 C CNN
+F 0 "#PWR023" H 7400 5650 50  0001 C CNN
 F 1 "VCC" H 7400 5950 50  0000 C CNN
 F 2 "" H 7400 5800 50  0001 C CNN
@@
 $EndComp
 $Comp
-L VCC #PWR?
+L VCC #PWR024
 U 1 1 5BAADC63
 P 4400 1450
-F 0 "#PWR?" H 4400 1300 50  0001 C CNN
+F 0 "#PWR024" H 4400 1300 50  0001 C CNN
 F 1 "VCC" H 4400 1600 50  0000 C CNN
 F 2 "" H 4400 1450 50  0001 C CNN
@@
 $EndComp
 $Comp
-L VCC #PWR?
+L VCC #PWR025
 U 1 1 5BAADD9C
 P 5150 2350
-F 0 "#PWR?" H 5150 2200 50  0001 C CNN
+F 0 "#PWR025" H 5150 2200 50  0001 C CNN
 F 1 "VCC" H 5150 2500 50  0000 C CNN
 F 2 "" H 5150 2350 50  0001 C CNN
@@
 F 0 "R_USB1" V 4650 2450 50  0000 C CNN
 F 1 "22" V 4750 2450 50  0000 C CNN
-F 2 "" H 4750 2450 60  0000 C CNN
+F 2 "Resistors_SMD:R_0805_HandSoldering" H 4750 2450 60  0001 C CNN
 F 3 "" H 4750 2450 60  0000 C CNN
 	1    4750 2450
@@
 F 0 "R_USB2" V 4830 2550 50  0000 C CNN
 F 1 "22" V 4750 2550 50  0000 C CNN
-F 2 "" H 4750 2550 60  0000 C CNN
+F 2 "Resistors_SMD:R_0805_HandSoldering" H 4750 2550 60  0001 C CNN
 F 3 "" H 4750 2550 60  0000 C CNN
 	1    4750 2550
@@
 	4200 2750 4200 3200
 $Comp
-L VCC #PWR?
+L VCC #PWR026
 U 1 1 5BAB3C15
 P 5150 2850
-F 0 "#PWR?" H 5150 2700 50  0001 C CNN
+F 0 "#PWR026" H 5150 2700 50  0001 C CNN
 F 1 "VCC" H 5150 3000 50  0000 C CNN
 F 2 "" H 5150 2850 50  0001 C CNN
@@
 F 0 "C_VBUS1" H 5650 6100 50  0000 L CNN
 F 1 "10u" H 5650 5900 50  0000 L CNN
-F 2 "" H 5600 6000 60  0000 C CNN
+F 2 "Capacitors_SMD:C_0805_HandSoldering" H 5600 6000 60  0001 C CNN
 F 3 "" H 5600 6000 60  0000 C CNN
 	1    5600 6000
@@
 $EndComp
 $Comp
-L VCC #PWR?
+L VCC #PWR027
 U 1 1 5BAB451B
 P 4200 4700
-F 0 "#PWR?" H 4200 4550 50  0001 C CNN
+F 0 "#PWR027" H 4200 4550 50  0001 C CNN
 F 1 "VCC" H 4200 4850 50  0000 C CNN
 F 2 "" H 4200 4700 50  0001 C CNN
@@
 $EndComp
 $Comp
-L GND #PWR?
+L GND #PWR028
 U 1 1 5BAB46A3
 P 5600 6200
-F 0 "#PWR?" H 5600 5950 50  0001 C CNN
+F 0 "#PWR028" H 5600 5950 50  0001 C CNN
 F 1 "GND" H 5600 6050 50  0000 C CNN
 F 2 "" H 5600 6200 50  0001 C CNN
@@
 	4050 4700 4200 4700
 $Comp
-L VCC #PWR?
+L VCC #PWR029
 U 1 1 5BAB5080
 P 5600 5800
-F 0 "#PWR?" H 5600 5650 50  0001 C CNN
+F 0 "#PWR029" H 5600 5650 50  0001 C CNN
 F 1 "VCC" H 5600 5950 50  0000 C CNN
 F 2 "" H 5600 5800 50  0001 C CNN

Commit message: 2018.10.02 Nightly
Parts:
- C_AREF1, C_AVCC1, C_CLK1, C_CLK2, C_UCAP1, C_UVCC1, C_VBUS1, C_VCC1, C_VCC2: symbol C -> keyboard_parts:C
- R_HWB1, R_RST1, R_USB1, R_USB2: symbol R -> keyboard_parts:R
- SW1: symbol SW_PUSH -> keyboard_parts:SW_PUSH
- U1: symbol AT90USB1286-AU -> jay:AT90USB1286-AU
- Y1: symbol Crystal_GND24 -> Device:Crystal_GND24
Connections:
- wire segments 46 -> 49
Changed lines of the file:
@@
-EESchema Schematic File Version 2
-LIBS:keyboard_parts
-LIBS:jay
-LIBS:power
-LIBS:device
-LIBS:transistors
-LIBS:conn
-LIBS:linear
-LIBS:regul
-LIBS:74xx
-LIBS:cmos4000
-LIBS:adc-dac
-LIBS:memory
-LIBS:xilinx
-LIBS:microcontrollers
-LIBS:dsp
-LIBS:microchip
-LIBS:analog_switches
-LIBS:motorola
-LIBS:texas
-LIBS:intel
-LIBS:audio
-LIBS:interface
-LIBS:digital-audio
-LIBS:philips
-LIBS:display
-LIBS:cypress
-LIBS:siliconi
-LIBS:opto
-LIBS:atmel
-LIBS:contrib
-LIBS:valves
-LIBS:JayKey1-cache
-EELAYER 25 0
+EESchema Schematic File Version 4
+EELAYER 26 0
 EELAYER END
 $Descr A4 11693 8268
@@
 Title "JayKey1 Schematic"
 Date ""
-Rev "1.1 (180427)"
+Rev "1.2 (???)"
 Comp "Josue Galeas"
 Comment1 ""
@@
 col13
 $Comp
-L C C_CLK1
+L keyboard_parts:C C_CLK1
 U 1 1 5A0B3A8B
 P 3350 2700
@@
 $EndComp
 $Comp
-L C C_CLK2
+L keyboard_parts:C C_CLK2
 U 1 1 5A0B3AC7
 P 3850 2700
@@
 $EndComp
 $Comp
-L GND #PWR01
+L power:GND #PWR01
 U 1 1 5A0B3FFB
 P 3600 2200
@@
 $EndComp
 $Comp
-L GND #PWR02
+L power:GND #PWR02
 U 1 1 5A0B403C
 P 3350 2900
@@
 $EndComp
 $Comp
-L GND #PWR03
+L power:GND #PWR03
 U 1 1 5A0B406B
 P 3850 2900
@@
 $EndComp
 $Comp
-L GND #PWR04
+L power:GND #PWR04
 U 1 1 5A0B42A8
 P 3600 2600
@@
 $EndComp
 $Comp
-L C C_AREF1
+L keyboard_parts:C C_AREF1
 U 1 1 5A0B4C67
 P 4500 3400
@@
 $EndComp
 $Comp
-L GND #PWR05
+L power:GND #PWR05
 U 1 1 5A0B4CA7
 P 4500 3600
@@
 $EndComp
 $Comp
-L GND #PWR06
+L power:GND #PWR06
 U 1 1 5A0B4F28
 P 6400 5350
@@
 $EndComp
 $Comp
-L GND #PWR07
+L power:GND #PWR07
 U 1 1 5A0B4F5A
 P 6500 5350
@@
 $EndComp
 $Comp
-L GND #PWR08
+L power:GND #PWR08
 U 1 1 5A0B4F8C
 P 6600 5350
@@
 $EndComp
 $Comp
-L GND #PWR09
+L power:GND #PWR09
 U 1 1 5A0B5542
 P 5150 2650
@@
 $EndComp
 $Comp
-L C C_UCAP1
+L keyboard_parts:C C_UCAP1
 U 1 1 5A0B5574
 P 4200 3400
@@
 $EndComp
 $Comp
-L GND #PWR010
+L power:GND #PWR010
 U 1 1 5A0B55F6
 P 4200 3600
@@
 $EndComp
 $Comp
-L R R_HWB1
+L keyboard_parts:R R_HWB1
 U 1 1 5A0B605B
 P 4800 4850
@@
 $EndComp
 $Comp
-L GND #PWR011
+L power:GND #PWR011
 U 1 1 5A0B60A2
 P 4800 5100
@@
 $EndComp
 $Comp
-L C C_UVCC1
+L keyboard_parts:C C_UVCC1
 U 1 1 5A0B6D57
 P 6050 6000
@@
 $EndComp
 $Comp
-L GND #PWR012
+L power:GND #PWR012
 U 1 1 5A0B6DE3
 P 6050 6200
@@
 $EndComp
 $Comp
-L C C_VCC1
+L keyboard_parts:C C_VCC1
 U 1 1 5A0B6FCB
 P 6500 6000
@@
 $EndComp
 $Comp
-L C C_VCC2
+L keyboard_parts:C C_VCC2
 U 1 1 5A0B70AE
 P 6950 6000
@@
 $EndComp
 $Comp
-L C C_AVCC1
+L keyboard_parts:C C_AVCC1
 U 1 1 5A0B7168
 P 7400 6000
@@
 $EndComp
 $Comp
-L GND #PWR013
+L power:GND #PWR013
 U 1 1 5A0B71F2
 P 6500 6200
@@
 $EndComp
 $Comp
-L GND #PWR014
+L power:GND #PWR014
 U 1 1 5A0B7236
 P 6950 6200
@@
 $EndComp
 $Comp
-L GND #PWR015
+L power:GND #PWR015
 U 1 1 5A0B727A
 P 7400 6200
@@
 $EndComp
 $Comp
-L R R_RST1
+L keyboard_parts:R R_RST1
 U 1 1 5A0B7D8A
 P 4650 1450
@@
 $EndComp
 $Comp
-L SW_PUSH SW1
+L keyboard_parts:SW_PUSH SW1
 U 1 1 5A0B7EDF
 P 4650 1750
@@
 $EndComp
 $Comp
-L GND #PWR016
+L power:GND #PWR016
 U 1 1 5A0B8008
 P 4350 1750
@@
 $EndComp
 $Comp
-L Crystal_GND24 Y1
+L Device:Crystal_GND24 Y1
 U 1 1 5A0E38FE
 P 3600 2400
@@
 DPLUS
 $Comp
-L AT90USB1286-AU U1
+L jay:AT90USB1286-AU U1
 U 1 1 5BA7F9F5
 P 6500 3400
@@
 	4800 4250 4900 4150
 Wire Wire Line
-	4950 1750 5150 1750
+	4950 1750 5050 1750
 Wire Wire Line
 	4900 1450 5050 1450
@@
 Connection ~ 5050 1750
 Wire Wire Line
-	3850 2100 3850 2500
-Wire Wire Line
-	3350 2000 3350 2500
+	3850 2100 3850 2400
+Wire Wire Line
+	3350 2000 3350 2400
 Wire Wire Line
 	7850 2050 8100 2050
@@
 Wire Wire Line
 	7850 2450 8100 2450
-Wire Bus Line
-	8200 2150 8200 2650
 Wire Bus Line
 	8200 2650 8350 2650
@@
 NoConn ~ 5150 5000
 Wire Bus Line
-	8200 3550 8200 5200
-Wire Bus Line
 	8200 5200 8350 5200
 Text Label 8350 5200 0    60   ~ 0
 col[00:20]
-Wire Bus Line
-	4800 3550 4800 4350
 Wire Bus Line
 	4800 4350 4650 4350
@@
 DPLUS
 $Comp
-L VCC #PWR017
+L power:VCC #PWR017
 U 1 1 5BAAD93C
 P 6400 1400
@@
 $EndComp
 $Comp
-L VCC #PWR018
+L power:VCC #PWR018
 U 1 1 5BAAD9A4
 P 6500 1400
@@
 $EndComp
 $Comp
-L VCC #PWR019
+L power:VCC #PWR019
 U 1 1 5BAADA0C
 P 6600 1400
@@
 $EndComp
 $Comp
-L VCC #PWR020
+L power:VCC #PWR020
 U 1 1 5BAADA98
 P 6050 5800
@@
 $EndComp
 $Comp
-L VCC #PWR021
+L power:VCC #PWR021
 U 1 1 5BAADB00
 P 6500 5800
@@
 $EndComp
 $Comp
-L VCC #PWR022
+L power:VCC #PWR022
 U 1 1 5BAADB68
 P 6950 5800
@@
 $EndComp
 $Comp
-L VCC #PWR023
+L power:VCC #PWR023
 U 1 1 5BAADBD0
 P 7400 5800
@@
 $EndComp
 $Comp
-L VCC #PWR024
+L power:VCC #PWR024
 U 1 1 5BAADC63
 P 4400 1450
@@
 $EndComp
 $Comp
-L VCC #PWR025
+L power:VCC #PWR025
 U 1 1 5BAADD9C
 P 5150 2350
@@
 $EndComp
 $Comp
-L R R_USB1
+L keyboard_parts:R R_USB1
 U 1 1 5BAAF9D4
 P 4750 2450
@@
 $EndComp
 $Comp
-L R R_USB2
+L keyboard_parts:R R_USB2
 U 1 1 5BAAFAA2
 P 4750 2550
@@
 	4200 2750 4200 3200
 $Comp
-L VCC #PWR026
+L power:VCC #PWR026
 U 1 1 5BAB3C15
 P 5150 2850
@@
 $EndComp
 $Comp
-L C C_VBUS1
+L keyboard_parts:C C_VBUS1
 U 1 1 5BAB4287
 P 5600 6000
@@
 $EndComp
 $Comp
-L VCC #PWR027
+L power:VCC #PWR027
 U 1 1 5BAB451B
 P 4200 4700
@@
 $EndComp
 $Comp
-L GND #PWR028
+L power:GND #PWR028
 U 1 1 5BAB46A3
 P 5600 6200
@@
 	4050 4700 4200 4700
 $Comp
-L VCC #PWR029
+L power:VCC #PWR029
 U 1 1 5BAB5080
 P 5600 5800
@@
 	1    0    0    -1
 $EndComp
+Wire Wire Line
+	5050 1750 5150 1750
+Wire Wire Line
+	3850 2400 3850 2500
+Wire Wire Line
+	3350 2400 3350 2500
+Wire Bus Line
+	8200 2150 8200 2650
+Wire Bus Line
+	4800 3550 4800 4350
+Wire Bus Line
+	8200 3550 8200 5200
 $EndSCHEMATC

Commit message: 2018.10.25 Nightly
Parts:
- SW1: footprint Buttons_Switches_SMD:SW_SPST_TL3342 -> Button_Switch_SMD:SW_SPST_TL3342
- U1: footprint Housings_QFP:TQFP-64_14x14mm_Pitch0.8mm -> Package_QFP:TQFP-64_14x14mm_P0.8mm
- Y1: footprint Crystals:Crystal_SMD_SeikoEpson_FA238-4pin_3.2x2.5mm -> Crystal:Crystal_SMD_SeikoEpson_FA238-4Pin_3.2x2.5mm_HandSoldering
Changed lines of the file:
@@
 F 0 "SW1" H 4800 1860 50  0000 C CNN
 F 1 "SW_PUSH" H 4650 1670 50  0000 C CNN
-F 2 "Buttons_Switches_SMD:SW_SPST_TL3342" H 4650 1750 60  0001 C CNN
+F 2 "Button_Switch_SMD:SW_SPST_TL3342" H 4650 1750 60  0001 C CNN
 F 3 "" H 4650 1750 60  0000 C CNN
 	1    4650 1750
@@
 F 0 "Y1" H 3650 2600 50  0000 L CNN
 F 1 "16M" H 3650 2200 50  0000 L CNN
-F 2 "Crystals:Crystal_SMD_SeikoEpson_FA238-4pin_3.2x2.5mm" H 3600 2400 50  0001 C CNN
+F 2 "Crystal:Crystal_SMD_SeikoEpson_FA238-4Pin_3.2x2.5mm_HandSoldering" H 3600 2400 50  0001 C CNN
 F 3 "" H 3600 2400 50  0001 C CNN
 	1    3600 2400
@@
 F 0 "U1" H 5400 5250 60  0000 C CNN
 F 1 "AT90USB1286-AU" H 7250 1600 60  0000 C CNN
-F 2 "Housings_QFP:TQFP-64_14x14mm_Pitch0.8mm" H 5600 2900 60  0001 C CNN
+F 2 "Package_QFP:TQFP-64_14x14mm_P0.8mm" H 5600 2900 60  0001 C CNN
 F 3 "" H 5600 2900 60  0001 C CNN
 	1    6500 3400

Commit message: 2018.11.29 Nightly
Parts:
- C_AREF1, C_AVCC1, C_CLK1, C_CLK2, C_UCAP1, C_UVCC1, C_VBUS1, C_VCC1, C_VCC2: footprint Capacitors_SMD:C_0805_HandSoldering -> Capacitor_SMD:C_0805_2012Metric_Pad1.15x1.40mm_HandSolder
- R_HWB1, R_RST1, R_USB1, R_USB2: footprint Resistors_SMD:R_0805_HandSoldering -> Resistor_SMD:R_0805_2012Metric_Pad1.15x1.40mm_HandSolder
Connections:
- net labels removed: col[00:20], row[0:4]
- wire segments 49 -> 23
Other:
- moved on the sheet: C_AREF1, C_AVCC1, C_CLK1, C_CLK2, C_UCAP1, C_UVCC1, C_VBUS1, C_VCC1, C_VCC2, R_HWB1, R_RST1, R_USB1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
