File: PCB/JayKey1.sch (KiCad schematic (older format))
At the start: 16 parts, among them SW1 SW_PUSH, U1 AT90USB1286-AU, Y1 16M

Commit message: 2018.12.04 Nightly
Connections:
- net labels added: CLK_N, CLK_P, D_+, D_-, D_N, D_P
- net labels removed: DMINUS, DPLUS
Other:
- moved on the sheet: R_USB1, R_USB2
Changed lines of the file:
@@
 Title "JayKey1 Schematic"
 Date ""
-Rev "1.2 (???)"
+Rev "2.0 (???)"
 Comp "Josue Galeas"
 Comment1 ""
@@
 F27 "COL20" B R 9450 3950 60
 $EndSheet
-Text Label 4150 3150 2    60   ~ 0
-DMINUS
-Text Label 4150 3250 2    60   ~ 0
-DPLUS
+Text Label 4000 3150 2    60   ~ 0
+D_N
+Text Label 4000 3250 2    60   ~ 0
+D_P
 $Comp
 L jay:AT90USB1286-AU U1
@@
 	9600 5700 9450 5700
 Text Label 9600 5550 0    60   ~ 0
-DMINUS
+D_N
 Text Label 9600 5700 0    60   ~ 0
-DPLUS
+D_P
 $Comp
 L power:VCC #PWR017
@@
 L keyboard_parts:R R_USB1
 U 1 1 5BAAF9D4
-P 4400 3150
-F 0 "R_USB1" V 4300 3150 50  0000 C CNN
-F 1 "22" V 4400 3150 50  0000 C CNN
-F 2 "Resistor_SMD:R_0805_2012Metric_Pad1.15x1.40mm_HandSolder" H 4400 3150 60  0001 C CNN
-F 3 "" H 4400 3150 60  0000 C CNN
-	1    4400 3150
+P 4250 3150
+F 0 "R_USB1" V 4150 3150 50  0000 C CNN
+F 1 "22" V 4250 3150 50  0000 C CNN
+F 2 "Resistor_SMD:R_0805_2012Metric_Pad1.15x1.40mm_HandSolder" H 4250 3150 60  0001 C CNN
+F 3 "" H 4250 3150 60  0000 C CNN
+	1    4250 3150
 	0    1    1    0
 $EndComp
@@
 L keyboard_parts:R R_USB2
 U 1 1 5BAAFAA2
-P 4400 3250
-F 0 "R_USB2" V 4480 3250 50  0000 C CNN
-F 1 "22" V 4400 3250 50  0000 C CNN
-F 2 "Resistor_SMD:R_0805_2012Metric_Pad1.15x1.40mm_HandSolder" H 4400 3250 60  0001 C CNN
-F 3 "" H 4400 3250 60  0000 C CNN
-	1    4400 3250
+P 4250 3250
+F 0 "R_USB2" V 4330 3250 50  0000 C CNN
+F 1 "22" V 4250 3250 50  0000 C CNN
+F 2 "Resistor_SMD:R_0805_2012Metric_Pad1.15x1.40mm_HandSolder" H 4250 3250 60  0001 C CNN
+F 3 "" H 4250 3250 60  0000 C CNN
+	1    4250 3250
 	0    1    1    0
 $EndComp
-Wire Wire Line
-	4650 3150 4800 3150
-Wire Wire Line
-	4650 3250 4800 3250
 Wire Wire Line
 	4300 3800 4300 3900
@@
 Text Label 9450 3950 0    60   ~ 0
 col20
+Text Label 3000 3100 2    60   ~ 0
+CLK_P
+Text Label 3500 3100 0    60   ~ 0
+CLK_N
+Wire Wire Line
+	4500 3150 4800 3150
+Wire Wire Line
+	4500 3250 4800 3250
+Text Label 4550 3150 1    60   ~ 0
+D_-
+Text Label 4550 3250 3    60   ~ 0
+D_+
 $EndSCHEMATC

Commit message: 2018.12.14 Nightly 2
Connections:
- wire segments 23 -> 20
Other:
- moved on the sheet: C_CLK1, C_CLK2, R_USB1, R_USB2, Y1
Changed lines of the file:
@@
 L keyboard_parts:C C_CLK1
 U 1 1 5A0B3A8B
-P 3000 3400
-F 0 "C_CLK1" H 2700 3500 50  0000 L CNN
-F 1 "22p" H 2850 3300 50  0000 L CNN
-F 2 "Capacitor_SMD:C_0805_2012Metric_Pad1.15x1.40mm_HandSolder" H 3000 3400 60  0001 C CNN
-F 3 "" H 3000 3400 60  0000 C CNN
-	1    3000 3400
+P 2700 3400
+F 0 "C_CLK1" H 2400 3500 50  0000 L CNN
+F 1 "22p" H 2550 3300 50  0000 L CNN
+F 2 "Capacitor_SMD:C_0805_2012Metric_Pad1.15x1.40mm_HandSolder" H 2700 3400 60  0001 C CNN
+F 3 "" H 2700 3400 60  0000 C CNN
+	1    2700 3400
 	1    0    0    -1
 $EndComp
@@
 L keyboard_parts:C C_CLK2
 U 1 1 5A0B3AC7
-P 3500 3400
-F 0 "C_CLK2" H 3550 3500 50  0000 L CNN
-F 1 "22p" H 3550 3300 50  0000 L CNN
-F 2 "Capacitor_SMD:C_0805_2012Metric_Pad1.15x1.40mm_HandSolder" H 3500 3400 60  0001 C CNN
-F 3 "" H 3500 3400 60  0000 C CNN
-	1    3500 3400
+P 3200 3400
+F 0 "C_CLK2" H 3250 3500 50  0000 L CNN
+F 1 "22p" H 3250 3300 50  0000 L CNN
+F 2 "Capacitor_SMD:C_0805_2012Metric_Pad1.15x1.40mm_HandSolder" H 3200 3400 60  0001 C CNN
+F 3 "" H 3200 3400 60  0000 C CNN
+	1    3200 3400
 	1    0    0    -1
 $EndComp
@@
 L power:GND #PWR01
 U 1 1 5A0B3FFB
-P 3250 2900
-F 0 "#PWR01" H 3250 2650 50  0001 C CNN
-F 1 "GND" H 3250 2750 50  0000 C CNN
-F 2 "" H 3250 2900 50  0001 C CNN
-F 3 "" H 3250 2900 50  0001 C CNN
-	1    3250 2900
+P 2950 2900
+F 0 "#PWR01" H 2950 2650 50  0001 C CNN
+F 1 "GND" H 2950 2750 50  0000 C CNN
+F 2 "" H 2950 2900 50  0001 C CNN
+F 3 "" H 2950 2900 50  0001 C CNN
+	1    2950 2900
 	-1   0    0    1
 $EndComp
@@
 L power:GND #PWR02
 U 1 1 5A0B403C
-P 3000 3600
-F 0 "#PWR02" H 3000 3350 50  0001 C CNN
-F 1 "GND" H 3000 3450 50  0000 C CNN
-F 2 "" H 3000 3600 50  0001 C CNN
-F 3 "" H 3000 3600 50  0001 C CNN
-	1    3000 3600
+P 2700 3600
+F 0 "#PWR02" H 2700 3350 50  0001 C CNN
+F 1 "GND" H 2700 3450 50  0000 C CNN
+F 2 "" H 2700 3600 50  0001 C CNN
+F 3 "" H 2700 3600 50  0001 C CNN
+	1    2700 3600
 	1    0    0    -1
 $EndComp
@@
 L power:GND #PWR03
 U 1 1 5A0B406B
-P 3500 3600
-F 0 "#PWR03" H 3500 3350 50  0001 C CNN
-F 1 "GND" H 3500 3450 50  0000 C CNN
-F 2 "" H 3500 3600 50  0001 C CNN
-F 3 "" H 3500 3600 50  0001 C CNN
-	1    3500 3600
+P 3200 3600
+F 0 "#PWR03" H 3200 3350 50  0001 C CNN
+F 1 "GND" H 3200 3450 50  0000 C CNN
+F 2 "" H 3200 3600 50  0001 C CNN
+F 3 "" H 3200 3600 50  0001 C CNN
+	1    3200 3600
 	1    0    0    -1
 $EndComp
@@
 L power:GND #PWR04
 U 1 1 5A0B42A8
-P 3250 3300
-F 0 "#PWR04" H 3250 3050 50  0001 C CNN
-F 1 "GND" H 3250 3150 50  0000 C CNN
-F 2 "" H 3250 3300 50  0001 C CNN
-F 3 "" H 3250 3300 50  0001 C CNN
-	1    3250 3300
+P 2950 3300
+F 0 "#PWR04" H 2950 3050 50  0001 C CNN
+F 1 "GND" H 2950 3150 50  0000 C CNN
+F 2 "" H 2950 3300 50  0001 C CNN
+F 3 "" H 2950 3300 50  0001 C CNN
+	1    2950 3300
 	1    0    0    -1
 $EndComp
@@
 L Device:Crystal_GND24 Y1
 U 1 1 5A0E38FE
-P 3250 3100
-F 0 "Y1" H 3300 3300 50  0000 L CNN
-F 1 "16M" H 3300 2900 50  0000 L CNN
-F 2 "Crystal:Crystal_SMD_SeikoEpson_FA238-4Pin_3.2x2.5mm_HandSoldering" H 3250 3100 50  0001 C CNN
-F 3 "" H 3250 3100 50  0001 C CNN
-	1    3250 3100
+P 2950 3100
+F 0 "Y1" H 3000 3300 50  0000 L CNN
+F 1 "16M" H 3000 2900 50  0000 L CNN
+F 2 "Crystal:Crystal_SMD_SeikoEpson_FA238-4Pin_3.2x2.5mm_HandSoldering" H 2950 3100 50  0001 C CNN
+F 3 "" H 2950 3100 50  0001 C CNN
+	1    2950 3100
 	1    0    0    -1
 $EndComp
@@
 F27 "COL20" B R 9450 3950 60
 $EndSheet
-Text Label 4000 3150 2    60   ~ 0
+Text Label 3850 3150 2    60   ~ 0
 D_N
-Text Label 4000 3250 2    60   ~ 0
+Text Label 3850 3250 2    60   ~ 0
 D_P
 $Comp
@@
 Connection ~ 4700 2450
 Wire Wire Line
-	3500 2800 3500 3100
-Wire Wire Line
-	3000 2700 3000 3100
+	3200 2800 3200 3100
+Wire Wire Line
+	2700 2700 2700 3100
 NoConn ~ 4800 5000
 NoConn ~ 4800 5100
@@
 NoConn ~ 4800 5700
 Wire Wire Line
-	3400 3100 3500 3100
-Connection ~ 3500 3100
-Wire Wire Line
-	3100 3100 3000 3100
-Connection ~ 3000 3100
-Wire Wire Line
-	3000 2700 4800 2700
-Wire Wire Line
-	3500 2800 4800 2800
+	3100 3100 3200 3100
+Connection ~ 3200 3100
+Wire Wire Line
+	2800 3100 2700 3100
+Connection ~ 2700 3100
 $Sheet
-S 8400 5250 1050 600
+S 8400 5400 1050 450
 U 5BA8C67B
 F0 "USB" 60
 F1 "usb.sch" 60
-F2 "VBUS" B R 9450 5400 60
 F3 "DMINUS" B R 9450 5550 60
 F4 "DPLUS" B R 9450 5700 60
 $EndSheet
-Wire Wire Line
-	9600 5550 9450 5550
-Wire Wire Line
-	9600 5700 9450 5700
-Text Label 9600 5550 0    60   ~ 0
+Text Label 9450 5550 0    60   ~ 0
 D_N
-Text Label 9600 5700 0    60   ~ 0
+Text Label 9450 5700 0    60   ~ 0
 D_P
 $Comp
@@
 L keyboard_parts:R R_USB1
 U 1 1 5BAAF9D4
-P 4250 3150
-F 0 "R_USB1" V 4150 3150 50  0000 C CNN
-F 1 "22" V 4250 3150 50  0000 C CNN
-F 2 "Resistor_SMD:R_0805_2012Metric_Pad1.15x1.40mm_HandSolder" H 4250 3150 60  0001 C CNN
-F 3 "" H 4250 3150 60  0000 C CNN
-	1    4250 3150
+P 4100 3150
+F 0 "R_USB1" V 4000 3150 50  0000 C CNN
+F 1 "22" V 4100 3150 50  0000 C CNN
+F 2 "Resistor_SMD:R_0805_2012Metric_Pad1.15x1.40mm_HandSolder" H 4100 3150 60  0001 C CNN
+F 3 "" H 4100 3150 60  0000 C CNN
+	1    4100 3150
 	0    1    1    0
 $EndComp
@@
 L keyboard_parts:R R_USB2
 U 1 1 5BAAFAA2
-P 4250 3250
-F 0 "R_USB2" V 4330 3250 50  0000 C CNN
-F 1 "22" V 4250 3250 50  0000 C CNN
-F 2 "Resistor_SMD:R_0805_2012Metric_Pad1.15x1.40mm_HandSolder" H 4250 3250 60  0001 C CNN
-F 3 "" H 4250 3250 60  0000 C CNN
-	1    4250 3250
+P 4100 3250
+F 0 "R_USB2" V 4180 3250 50  0000 C CNN
+F 1 "22" V 4100 3250 50  0000 C CNN
+F 2 "Resistor_SMD:R_0805_2012Metric_Pad1.15x1.40mm_HandSolder" H 4100 3250 60  0001 C CNN
+F 3 "" H 4100 3250 60  0000 C CNN
+	1    4100 3250
 	0    1    1    0
 $EndComp
@@
 $EndComp
 $Comp
-L power:VCC #PWR027
-U 1 1 5BAB451B
-P 9600 5400
-F 0 "#PWR027" H 9600 5250 50  0001 C CNN
-F 1 "VCC" H 9600 5550 50  0000 C CNN
-F 2 "" H 9600 5400 50  0001 C CNN
-F 3 "" H 9600 5400 50  0001 C CNN
-	1    9600 5400
-	0    1    1    0
-$EndComp
-$Comp
 L power:GND #PWR028
 U 1 1 5BAB46A3
@@
 	1    0    0    -1
 $EndComp
-Wire Wire Line
-	9450 5400 9600 5400
 $Comp
 L power:VCC #PWR029
@@
 	4700 2450 4800 2450
 Wire Wire Line
-	3500 3100 3500 3200
-Wire Wire Line
-	3000 3100 3000 3200
+	3200 3100 3200 3200
+Wire Wire Line
+	2700 3100 2700 3200
 Wire Wire Line
 	4600 5200 4800 5200
@@
 Text Label 9450 3950 0    60   ~ 0
 col20
-Text Label 3000 3100 2    60   ~ 0
+Text Label 2700 3100 2    60   ~ 0
 CLK_P
-Text Label 3500 3100 0    60   ~ 0
+Text Label 3200 3100 0    60   ~ 0
 CLK_N
-Wire Wire Line
-	4500 3150 4800 3150
-Wire Wire Line
-	4500 3250 4800 3250
-Text Label 4550 3150 1    60   ~ 0
+Text Label 4350 3150 0    60   ~ 0
 D_-
-Text Label 4550 3250 3    60   ~ 0
+Text Label 4350 3250 0    60   ~ 0
 D_+
+Wire Wire Line
+	2700 2700 4800 2700
+Wire Wire Line
+	3200 2800 4800 2800
+Wire Wire Line
+	4350 3150 4800 3150
+Wire Wire Line
+	4350 3250 4800 3250
 $EndSCHEMATC
