File: PCB/key_matrix.sch (KiCad schematic (older format))
At the start: 186 parts, among them K0,0 KEYSW, K0,1 KEYSW, K0,10 KEYSW, K0,11 KEYSW, K0,12 KEYSW, K0,13 KEYSW, K0,14 KEYSW, K0,15 KEYSW, K0,16 KEYSW, K0,17 KEYSW, K0,18 KEYSW, K0,19 KEYSW, K0,2 KEYSW, K0,20 KEYSW, K0,3 KEYSW, K0,4 KEYSW, K0,5 KEYSW, K0,6 KEYSW, K0,7 KEYSW, K0,8 KEYSW, K0,9 KEYSW, K1,0 KEYSW, K1,1 KEYSW, K1,10 KEYSW, K1,11 KEYSW, K1,12 KEYSW, K1,13 KEYSW, K1,14 KEYSW, K1,15 KEYSW, K1,16 KEYSW, K1,17 KEYSW, K1,18 KEYSW, K1,19 KEYSW, K1,2 KEYSW, K1,20 KEYSW, K1,3 KEYSW, K1,4 KEYSW, K1,5 KEYSW, K1,6 KEYSW, K1,7 KEYSW, K1,8 KEYSW, K1,9 KEYSW, K2,0 KEYSW, K2,1 KEYSW, K2,10 KEYSW, K2,11 KEYSW, K2,12 KEYSW, K2,13 KEYSW, K2,14 KEYSW, K2,15 KEYSW, K2,17 KEYSW, K2,18 KEYSW, K2,19 KEYSW, K2,2 KEYSW, K2,20 KEYSW, K2,4 KEYSW, K2,5 KEYSW, K2,6 KEYSW, K2,7 KEYSW, K2,8 KEYSW, K2,9 KEYSW, K3,0 KEYSW, K3,1 KEYSW, K3,10 KEYSW, K3,11 KEYSW, K3,12 KEYSW, K3,13 KEYSW, K3,14 KEYSW, K3,16 KEYSW, K3,18 KEYSW, K3,19 KEYSW, K3,2 KEYSW, K3,20 KEYSW, K3,3 KEYSW, K3,4 KEYSW, K3,5 KEYSW, K3,6 KEYSW, K3,7 KEYSW, K3,8 KEYSW, K3,9 KEYSW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

Commit message: 2018.10.02 Nightly
Parts:
- D0,0, D0,1, D0,10, D0,11, D0,12, D0,13, D0,14, D0,15, D0,16, D0,17, D0,18, D0,19, D0,2, D0,20, D0,3, D0,4, D0,5, D0,6, D0,7, D0,8, D0,9, D1,0, D1,1, D1,10, D1,11, D1,12, D1,13, D1,14, D1,15, D1,16, D1,17, D1,18, D1,19, D1,2, D1,20, D1,3, D1,4, D1,5, D1,6, D1,7, D1,8, D1,9, D2,0, D2,1, D2,10, D2,11, D2,12, D2,13, D2,14, D2,15, D2,17, D2,18, D2,19, D2,2, D2,20, D2,4, D2,5, D2,6, D2,7, D2,8, D2,9, D3,0, D3,1, D3,10, D3,11, D3,12, D3,13, D3,14, D3,16, D3,18, D3,19, D3,2, D3,20, D3,3, D3,4, D3,5, D3,6, D3,7, D3,8, D3,9, D4,0, D4,13, D4,14, D4,16, D4,17, D4,18, D4,19, D4,2, D4,20, D4,4, D4,5, D4,6, D4,9: symbol D -> keyboard_parts:D
- K0,0, K0,1, K0,10, K0,11, K0,12, K0,13, K0,14, K0,15, K0,16, K0,17, K0,18, K0,19, K0,2, K0,20, K0,3, K0,4, K0,5, K0,6, K0,7, K0,8, K0,9, K1,0, K1,1, K1,10, K1,11, K1,12, K1,13, K1,14, K1,15, K1,16, K1,17, K1,18, K1,19, K1,2, K1,20, K1,3, K1,4, K1,5, K1,6, K1,7, K1,8, K1,9, K2,0, K2,1, K2,10, K2,11, K2,12, K2,13, K2,14, K2,15, K2,17, K2,18, K2,19, K2,2, K2,20, K2,4, K2,5, K2,6, K2,7, K2,8, K2,9, K3,0, K3,1, K3,10, K3,11, K3,12, K3,13, K3,14, K3,16, K3,18, K3,19, K3,2, K3,20, K3,3, K3,4, K3,5, K3,6, K3,7, K3,8, K3,9, K4,0, K4,13, K4,14, K4,16, K4,17, K4,18, K4,19, K4,2, K4,20, K4,4, K4,5, K4,6, K4,9: symbol KEYSW -> keyboard_parts:KEYSW

Commit message: 2018.11.29 Nightly
Connections:
- net col00 renamed COL00
- net col01 renamed COL01
- net col02 renamed COL02
- net col03 renamed COL03
- net col04 renamed COL04
- net col05 renamed COL05
- net col06 renamed COL06
- net col07 renamed COL07
- net col08 renamed COL08
- net col09 renamed COL09
- net col10 renamed COL10
- net col11 renamed COL11
- net col12 renamed COL12
- net col13 renamed COL13
- net col14 renamed COL14
- net col15 renamed COL15
- net col16 renamed COL16
- net col17 renamed COL17
- net col18 renamed COL18
- net col19 renamed COL19
- net col20 renamed COL20
- net row0 renamed ROW0
- net row1 renamed ROW1
- net row2 renamed ROW2
- net row3 renamed ROW3
- net row4 renamed ROW4
Other:
- moved on the sheet: D0,0, D0,1, D0,10, D0,11, D0,12, D0,13, D0,14, D0,15, D0,16, D0,17, D0,18, D0,19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
