File: PCB/usb.sch (KiCad schematic (older format))
At the start: 16 parts

Commit message: 2018.09.25 Nightly
Parts:
- removed C_VBUS? (x2): 10u, Capacitors_SMD:C_0805_HandSoldering, symbol C
- removed D?: PESD5V0L2BT, symbol PESD5V0L2BT
- removed D_VBUS?: D, keyboard_parts:D_SOD123_axial, symbol D
- removed J?: USB_C_Receptacle, Connectors_USB:USB_C_Receptacle_Amphenol_12401610E4-2A, symbol USB_C_Receptacle
- removed R_USB? (x2): 5.1k, Resistors_SMD:R_0805_HandSoldering, symbol R
- removed R_USB? (x2): 22, Resistors_SMD:R_0805_HandSoldering, symbol R
- added D_ESD1: PESD5V0L2BT, TO_SOT_Packages_SMD:SOT-23, symbol PESD5V0L2BT
- added D_VBUS1: D, keyboard_parts:D_SOD123_axial, symbol D
- added J1: USB_C_Receptacle, Connectors_USB:USB_C_Receptacle_Amphenol_12401610E4-2A, symbol USB_C_Receptacle
- added R_USB1, R_USB2: 5.1k, Resistors_SMD:R_0805_HandSoldering, symbol R
- added R_USB3, R_USB4: 22, Resistors_SMD:R_0805_HandSoldering, symbol R
- D_ESD2: renamed from D?; footprint (none) -> TO_SOT_Packages_SMD:SOT-23
- gave numbers to parts that had none: 6
Connections:
- wire segments 39 -> 33
Other:
- moved on the sheet: D_VBUS2, J2, R_USB5, R_USB6, R_USB7, R_USB8

Commit message: 2018.09.29 Nightly
Parts:
- removed R_USB3, R_USB4, R_USB7, R_USB8: 22, Resistors_SMD:R_0805_HandSoldering, symbol R
- renumbered R_USB1 to R_USB3, R_USB2 to R_USB4
Connections:
- wire segments 33 -> 29
Other:
- moved on the sheet: D_VBUS1, D_VBUS2, J1, J2, R_USB3, R_USB4, R_USB5, R_USB6

Commit message: 2018.10.02 Nightly
Parts:
- removed J1, J2: USB_C_Receptacle, Connectors_USB:USB_C_Receptacle_Amphenol_12401610E4-2A, symbol USB_C_Receptacle
- added J1, J2: USB_C_Receptacle, Connector_USB:USB_C_Receptacle_Amphenol_12401610E4-2A, symbol Connector:USB_C_Receptacle
- D_ESD1, D_ESD2: symbol PESD5V0L2BT -> jay:PESD5V0L2BT
- D_VBUS1, D_VBUS2: symbol D -> keyboard_parts:D
- R_USB3, R_USB4, R_USB5, R_USB6: symbol R -> keyboard_parts:R
Connections:
- wire segments 29 -> 39
Changed lines of the file:
@@
-EESchema Schematic File Version 2
-LIBS:keyboard_parts
-LIBS:jay
-LIBS:power
-LIBS:device
-LIBS:transistors
-LIBS:conn
-LIBS:linear
-LIBS:regul
-LIBS:74xx
-LIBS:cmos4000
-LIBS:adc-dac
-LIBS:memory
-LIBS:xilinx
-LIBS:microcontrollers
-LIBS:dsp
-LIBS:microchip
-LIBS:analog_switches
-LIBS:motorola
-LIBS:texas
-LIBS:intel
-LIBS:audio
-LIBS:interface
-LIBS:digital-audio
-LIBS:philips
-LIBS:display
-LIBS:cypress
-LIBS:siliconi
-LIBS:opto
-LIBS:atmel
-LIBS:contrib
-LIBS:valves
-LIBS:JayKey1-cache
-EELAYER 25 0
+EESchema Schematic File Version 4
+EELAYER 26 0
 EELAYER END
 $Descr A4 11693 8268
@@
 Title "USB Schematic"
 Date ""
-Rev "1.1 (180427)"
+Rev "1.2 (???)"
 Comp "Josue Galeas"
 Comment1 ""
@@
 $EndDescr
 $Comp
-L USB_C_Receptacle J2
-U 1 1 5BA8D347
-P 4500 4000
-F 0 "J2" H 4100 5450 50  0000 L CNN
-F 1 "USB_C_Receptacle" H 4900 5450 50  0000 R CNN
-F 2 "Connectors_USB:USB_C_Receptacle_Amphenol_12401610E4-2A" H 4650 4000 50  0001 C CNN
-F 3 "" H 4650 4000 50  0001 C CNN
-	1    4500 4000
-	1    0    0    -1
-$EndComp
-$Comp
-L GND #PWR030
+L power:GND #PWR030
 U 1 1 5BA8D348
 P 4200 5600
@@
 $EndComp
 $Comp
-L GND #PWR031
+L power:GND #PWR031
 U 1 1 5BA8D349
 P 4300 5600
@@
 $EndComp
 $Comp
-L GND #PWR032
+L power:GND #PWR032
 U 1 1 5BA8D34A
 P 4400 5600
@@
 $EndComp
 $Comp
-L GND #PWR033
+L power:GND #PWR033
 U 1 1 5BA8D34B
 P 4500 5600
@@
 $EndComp
 $Comp
-L GND #PWR034
+L power:GND #PWR034
 U 1 1 5BA8D34C
 P 4600 5600
@@
 $EndComp
 $Comp
-L R R_USB6
+L keyboard_parts:R R_USB6
 U 1 1 5BA8D34D
 P 5350 3400
@@
 $EndComp
 $Comp
-L R R_USB5
+L keyboard_parts:R R_USB5
 U 1 1 5BA8D34E
 P 5350 3200
@@
 $EndComp
 $Comp
-L GND #PWR035
+L power:GND #PWR035
 U 1 1 5BA8D34F
 P 5600 3400
@@
 $EndComp
 $Comp
-L GND #PWR036
+L power:GND #PWR036
 U 1 1 5BA8D350
 P 5600 3200
@@
 Text Label 5600 2700 0    60   ~ 0
 VBUS
-Text Notes 4100 2500 0    60   ~ 0
+Text Notes 4250 2350 0    60   ~ 0
 Left USB Port
 $Comp
-L D D_VBUS2
+L keyboard_parts:D D_VBUS2
 U 1 1 5BA8D355
 P 5450 2700
@@
 DPLUS
 $Comp
-L PESD5V0L2BT D_ESD2
+L jay:PESD5V0L2BT D_ESD2
 U 1 1 5BA90EA0
 P 5700 4450
@@
 $EndComp
 $Comp
-L GND #PWR037
+L power:GND #PWR037
 U 1 1 5BAAAA06
 P 5700 5000
@@
 $EndComp
 Wire Wire Line
-	5100 3600 6000 3600
-Wire Wire Line
-	5100 3800 6000 3800
+	5100 3600 5900 3600
+Wire Wire Line
+	5100 3800 5500 3800
 Wire Wire Line
 	5200 3000 5100 3000
 Wire Wire Line
-	5200 2700 5200 3000
-Wire Wire Line
-	5100 2700 5300 2700
+	5200 2700 5200 2800
+Wire Wire Line
+	5100 2700 5200 2700
 Connection ~ 5200 2700
 Wire Wire Line
@@
 Connection ~ 5500 3800
 Connection ~ 5900 3600
-Wire Wire Line
-	5100 3300 5100 3400
-Wire Wire Line
-	5100 3500 5100 3600
-Wire Wire Line
-	5100 3700 5100 3800
-$Comp
-L USB_C_Receptacle J1
-U 1 1 5BAABDD0
-P 6850 4000
-F 0 "J1" H 6450 5450 50  0000 L CNN
-F 1 "USB_C_Receptacle" H 7250 5450 50  0000 R CNN
-F 2 "Connectors_USB:USB_C_Receptacle_Amphenol_12401610E4-2A" H 7000 4000 50  0001 C CNN
-F 3 "" H 7000 4000 50  0001 C CNN
-	1    6850 4000
-	1    0    0    -1
-$EndComp
-$Comp
-L GND #PWR038
+$Comp
+L power:GND #PWR038
 U 1 1 5BAABDD6
 P 6550 5600
@@
 $EndComp
 $Comp
-L GND #PWR039
+L power:GND #PWR039
 U 1 1 5BAABDDC
 P 6650 5600
@@
 $EndComp
 $Comp
-L GND #PWR040
+L power:GND #PWR040
 U 1 1 5BAABDE2
 P 6750 5600
@@
 $EndComp
 $Comp
-L GND #PWR041
+L power:GND #PWR041
 U 1 1 5BAABDE8
 P 6850 5600
@@
 $EndComp
 $Comp
-L GND #PWR042
+L power:GND #PWR042
 U 1 1 5BAABDEE
 P 6950 5600
@@
 $EndComp
 $Comp
-L R R_USB4
+L keyboard_parts:R R_USB4
 U 1 1 5BAABDF4
 P 7700 3400
@@
 $EndComp
 $Comp
-L R R_USB3
+L keyboard_parts:R R_USB3
 U 1 1 5BAABDFA
 P 7700 3200
@@
 $EndComp
 $Comp
-L GND #PWR043
+L power:GND #PWR043
 U 1 1 5BAABE00
 P 7950 3400
@@
 $EndComp
 $Comp
-L GND #PWR044
+L power:GND #PWR044
 U 1 1 5BAABE06
 P 7950 3200
@@
 Text Label 7950 2700 0    60   ~ 0
 VBUS
-Text Notes 6450 2500 0    60   ~ 0
+Text Notes 6600 2350 0    60   ~ 0
 Right USB Port
 $Comp
-L D D_VBUS1
+L keyboard_parts:D D_VBUS1
 U 1 1 5BAABE32
 P 7800 2700
@@
 $EndComp
 $Comp
-L PESD5V0L2BT D_ESD1
+L jay:PESD5V0L2BT D_ESD1
 U 1 1 5BAABE38
 P 8050 4450
@@
 $EndComp
 $Comp
-L GND #PWR045
+L power:GND #PWR045
 U 1 1 5BAABE3E
 P 8050 5000
@@
 $EndComp
 Wire Wire Line
-	7450 3600 8350 3600
-Wire Wire Line
-	7450 3800 8350 3800
+	7450 3600 8250 3600
+Wire Wire Line
+	7450 3800 7850 3800
 Wire Wire Line
 	7550 3000 7450 3000
 Wire Wire Line
-	7550 2700 7550 3000
-Wire Wire Line
-	7450 2700 7650 2700
+	7550 2700 7550 2800
+Wire Wire Line
+	7450 2700 7550 2700
 Connection ~ 7550 2700
 Wire Wire Line
@@
 Connection ~ 8250 3600
 Wire Wire Line
+	7850 2700 7950 2700
+Wire Wire Line
+	5500 2700 5600 2700
+Wire Wire Line
+	5200 2700 5300 2700
+Wire Wire Line
+	5200 2800 5200 2900
+Wire Wire Line
+	5200 2900 5200 3000
+Wire Wire Line
+	5500 3800 6000 3800
+Wire Wire Line
+	5900 3600 6000 3600
+Wire Wire Line
+	7550 2700 7650 2700
+Wire Wire Line
+	7550 2800 7550 2900
+Wire Wire Line
+	7550 2900 7550 3000
+Wire Wire Line
+	7850 3800 8350 3800
+Wire Wire Line
+	8250 3600 8350 3600
+$Comp
+L Connector:USB_C_Receptacle J2
+U 1 1 5BB1A09A
+P 4500 4000
+F 0 "J2" H 4605 5567 50  0000 C CNN
+F 1 "USB_C_Receptacle" H 4605 5476 50  0000 C CNN
+F 2 "Connector_USB:USB_C_Receptacle_Amphenol_12401610E4-2A" H 4650 4000 50  0001 C CNN
+F 3 "http://www.usb.org/developers/docs/usb_31_033017.zip" H 4650 4000 50  0001 C CNN
+	1    4500 4000
+	1    0    0    -1
+$EndComp
+$Comp
+L Connector:USB_C_Receptacle J1
+U 1 1 5BB1A1D8
+P 6850 4000
+F 0 "J1" H 6955 5567 50  0000 C CNN
+F 1 "USB_C_Receptacle" H 6955 5476 50  0000 C CNN
+F 2 "Connector_USB:USB_C_Receptacle_Amphenol_12401610E4-2A" H 7000 4000 50  0001 C CNN
+F 3 "http://www.usb.org/developers/docs/usb_31_033017.zip" H 7000 4000 50  0001 C CNN
+	1    6850 4000
+	1    0    0    -1
+$EndComp
+Wire Wire Line
+	5100 3300 5100 3400
+Wire Wire Line
+	5100 3500 5100 3600
+Connection ~ 5100 3600
+Wire Wire Line
+	5100 3700 5100 3800
+Connection ~ 5100 3800
+Wire Wire Line
 	7450 3300 7450 3400
 Wire Wire Line
 	7450 3500 7450 3600
+Connection ~ 7450 3600
 Wire Wire Line
 	7450 3700 7450 3800
-Wire Wire Line
-	7850 2700 7950 2700
-Wire Wire Line
-	5500 2700 5600 2700
+Connection ~ 7450 3800
 $EndSCHEMATC

Commit message: 2018.10.25 Nightly
Parts:
- removed J1, J2: USB_C_Receptacle, Connector_USB:USB_C_Receptacle_Amphenol_12401610E4-2A, symbol Connector:USB_C_Receptacle
- added J1, J2: USB_C_Receptacle_USB2.0, Connector_USB:USB_C_Receptacle_Amphenol_12401610E4-2A, symbol Connector:USB_C_Receptacle_USB2.0
- D_ESD1, D_ESD2: footprint TO_SOT_Packages_SMD:SOT-23 -> Package_TO_SOT_SMD:SOT-23_Handsoldering
Connections:
- wire segments 39 -> 23
- no-connect marks 20 -> 4
Other:
- moved on the sheet: D_VBUS1, D_VBUS2, R_USB3, R_USB4, R_USB5, R_USB6

Commit message: 2018.11.29 Nightly
Parts:
- R_USB3, R_USB4, R_USB5, R_USB6: footprint Resistors_SMD:R_0805_HandSoldering -> Resistor_SMD:R_0805_2012Metric_Pad1.15x1.40mm_HandSolder
Other:
- moved on the sheet: D_VBUS1, D_VBUS2, R_USB3, R_USB4, R_USB5, R_USB6

Commit message: 2018.12.04 Nightly
Parts:
- removed D_ESD2: PESD5V0L2BT, Package_TO_SOT_SMD:SOT-23_Handsoldering, symbol jay:PESD5V0L2BT
- removed D_VBUS2: D, keyboard_parts:D_SOD123_axial, symbol keyboard_parts:D
- removed J2: USB_C_Receptacle_USB2.0, Connector_USB:USB_C_Receptacle_Amphenol_12401610E4-2A, symbol Connector:USB_C_Receptacle_USB2.0
- removed R_USB5, R_USB6: 5.1k, Resistor_SMD:R_0805_2012Metric_Pad1.15x1.40mm_HandSolder, symbol keyboard_parts:R
Connections:
- wire segments 23 -> 10
- no-connect marks 4 -> 2
Other:
- note removed: "Left USB Port"
- note removed: "Right USB Port"
- moved on the sheet: D_VBUS1, R_USB3, R_USB4

Commit message: 2018.12.14 Nightly 2
Connections:
- net labels added: VCC
- net labels removed: VBUS
Changed lines of the file:
@@
 Comment4 ""
 $EndDescr
-Text HLabel 6550 2950 2    60   BiDi ~ 0
-VBUS
 Text HLabel 6550 3550 2    60   BiDi ~ 0
 DMINUS
@@
 Wire Wire Line
 	5650 2950 6250 2950
+$Comp
+L power:VCC #PWR?
+U 1 1 5C15AB5B
+P 6550 2950
+F 0 "#PWR?" H 6550 2800 50  0001 C CNN
+F 1 "VCC" V 6567 3078 50  0000 L CNN
+F 2 "" H 6550 2950 50  0001 C CNN
+F 3 "" H 6550 2950 50  0001 C CNN
+	1    6550 2950
+	0    1    1    0
+$EndComp
 $EndSCHEMATC
